Commit message: V0.2

File: tp1_robot/urdf/diffbot.xacro (robot description, xacro)
@@ -1,92 +1,91 @@
 <?xml version="1.0"?>
 <robot name="diffbot" xmlns:xacro="http://www.ros.org/wiki/xacro">
-  <!-- Parámetros reutilizables -->
-  <xacro:property name="chassis_mass" value="0.8"/>
-  <xacro:property name="chassis_length" value="0.195"/>
-  <xacro:property name="chassis_width" value="0.1"/>
-  <xacro:property name="chassis_height" value="0.05"/>
-  <xacro:property name="wheel_radius" value="0.035"/>
-  <xacro:property name="wheel_separation" value="0.08"/>
-  <!-- Incluir macros -->
-  <xacro:include filename="$(find tp1_robot)/urdf/inertial_macros.xacro"/>
-  <xacro:include filename="$(find tp1_robot)/urdf/motor.xacro"/>
-  <!-- Base del robot (chasis) -->
-  <link name="base_link">
-    <visual>
-      <origin xyz="0 0 0" rpy="0 0 0"/>
-      <geometry>
-        <mesh filename="file://$(find tp1_robot)/meshes/chassis.stl" scale="0.001 0.001 0.001"/>
-      </geometry>
-      <material name="silver"/>
-    </visual>
-    <collision>
-      <origin xyz="0 0 0" rpy="0 0 0"/>
-      <geometry>
-        <box size="${chassis_length} ${chassis_width} ${chassis_height}"/>
-      </geometry>
-    </collision>
-    <xacro:inertial_box mass="${chassis_mass}" x="${chassis_length}" y="${chassis_width}" z="${chassis_height}">
-      <origin xyz="0 0 0" rpy="0 0 0"/>
-    </xacro:inertial_box>
-  </link>
-  <!-- Ruedas -->
-  <xacro:macro name="wheel" params="prefix side">
-    <link name="${prefix}_wheel">
-      <visual>
-        <origin xyz="0 0 0" rpy="1.5708 0 0"/>
-        <geometry>
-          <cylinder radius="${wheel_radius}" length="0.025"/>
-        </geometry>
-        <material name="black"/>
-      </visual>
-      <collision>
-        <origin xyz="0 0 0" rpy="1.5708 0 0"/>
-        <geometry>
-          <cylinder radius="${wheel_radius}" length="0.025"/>
-        </geometry>
-      </collision>
-      <xacro:inertial_cylinder mass="0.15" length="0.025" radius="${wheel_radius}">
-        <origin xyz="0 0 0" rpy="0 0 0"/>
-      </xacro:inertial_cylinder>
+    <!-- Parámetros reutilizables -->
+    <xacro:property name="chassis_mass" value="0.8"/>
+    <xacro:property name="chassis_length" value="0.195"/>
+    <xacro:property name="chassis_width" value="0.1"/>
+    <xacro:property name="chassis_height" value="0.05"/>
+    <xacro:property name="wheel_radius" value="0.035"/>
+    <xacro:property name="wheel_separation" value="0.08"/> <!-- Separación media -->
+    <!-- Incluir macros -->
+    <xacro:include filename="$(find tp1_robot)/urdf/inertial_macros.xacro"/>
+    <xacro:include filename="$(find tp1_robot)/urdf/motor.xacro"/>
+    <!-- Base del robot -->
+    <link name="base_link">
+        <visual>
+            <origin xyz="0 0 0" rpy="0 0 0"/>
+            <geometry>
+                <mesh filename="file://$(find tp1_robot)/meshes/chassis.stl" scale="0.001 0.001 0.001"/>
+            </geometry>
+            <material name="silver"/>
+        </visual>
+        <collision>
+            <origin xyz="0 0 0" rpy="0 0 0"/>
+            <geometry>
+                <box size="${chassis_length} ${chassis_width} ${chassis_height}"/>
+            </geometry>
+        </collision>
+        <xacro:inertial_box mass="${chassis_mass}" x="${chassis_length}" y="${chassis_width}" z="${chassis_height}">
+            <origin xyz="0 0 0" rpy="0 0 0"/>
+        </xacro:inertial_box>
     </link>
-    <joint name="${prefix}_wheel_joint" type="continuous">
-      <parent link="base_link"/>
-      <child link="${prefix}_wheel"/>
-      <axis xyz="0 1 0"/>
-      <origin xyz="${chassis_length/2 - 0.035} ${side*wheel_separation} -0.025"/>
-    </joint>
-  </xacro:macro>
-  <!-- Instanciar ruedas -->
-  <xacro:wheel prefix="left" side="1"/>
-  <xacro:wheel prefix="right" side="-1"/>
-  <!-- Motores -->
-  <xacro:motor prefix="left" chassis_width="${chassis_width}" reflect="false"/>
-  <xacro:motor prefix="right" chassis_width="${chassis_width}" reflect="true"/>
-  <gazebo>
-    <plugin name="gazebo_ros_control" filename="libgazebo_ros_diff_drive.so">
-      <ros>
-        <namespace>/diffbot</namespace>
-      </ros>
-      <wheel_separation>${wheel_separation * 2}</wheel_separation>
-      <wheel_diameter>${wheel_radius * 2}</wheel_diameter>
-      <left_joint>left_wheel_joint</left_joint>
-      <right_joint>right_wheel_joint</right_joint>
-    </plugin>
-  </gazebo>
-  <!-- Configuración de ros2_control -->
-  <ros2_control name="diffbot_controller" type="system">
-    <hardware>
-      <plugin>gazebo_ros2_control/RobotHWSim</plugin>
-    </hardware>
-    <joint name="left_wheel_joint">
-      <command_interface name="velocity"/>
-      <state_interface name="position"/>
-      <state_interface name="velocity"/>
-    </joint>
-    <joint name="right_wheel_joint">
-      <command_interface name="velocity"/>
-      <state_interface name="position"/>
-      <state_interface name="velocity"/>
-    </joint>
-  </ros2_control>
+    <!-- Macro de ruedas -->
+    <xacro:macro name="wheel" params="prefix side">
+        <link name="${prefix}_wheel">
+            <visual>
+                <origin xyz="0 0 0" rpy="1.5708 0 0"/>
+                <geometry>
+                    <cylinder radius="${wheel_radius}" length="0.025"/>
+                </geometry>
+                <material name="black"/>
+            </visual>
+            <collision>
+                <origin xyz="0 0 0" rpy="1.5708 0 0"/>
+                <geometry>
+                    <cylinder radius="${wheel_radius}" length="0.025"/>
+                </geometry>
+            </collision>
+            <xacro:inertial_cylinder mass="0.15" length="0.025" radius="${wheel_radius}">
+                <origin xyz="0 0 0" rpy="0 0 0"/>
+            </xacro:inertial_cylinder>
+        </link>
+        <joint name="${prefix}_wheel_joint" type="continuous">
+            <parent link="base_link"/>
+            <child link="${prefix}_wheel"/>
+            <axis xyz="0 1 0"/>
+            <origin xyz="${chassis_length/2 - 0.035} ${side*wheel_separation} -0.025"/>
+        </joint>
+    </xacro:macro>
+    <!-- Instanciar ruedas -->
+    <xacro:wheel prefix="left" side="1"/>
+    <xacro:wheel prefix="right" side="-1"/>
+    <!-- Motores -->
+    <xacro:motor prefix="left" chassis_width="${chassis_width}" reflect="false"/>
+    <xacro:motor prefix="right" chassis_width="${chassis_width}" reflect="true"/>
+    <!-- Plugin de Gazebo -->
+    <gazebo>
+        <plugin name="gazebo_ros_control" filename="libgazebo_ros_diff_drive.so">
+            <ros><namespace>/diffbot</namespace></ros>
+            <wheel_separation>${wheel_separation * 2}</wheel_separation>
+            <wheel_diameter>${wheel_radius * 2}</wheel_diameter>
+            <left_joint>left_wheel_joint</left_joint>
+            <right_joint>right_wheel_joint</right_joint>
+        </plugin>
+    </gazebo>
+    <!-- Configuración de ros2_control -->
+    <ros2_control name="diffbot_controller" type="system">
+        <hardware>
+            <plugin>gazebo_ros2_control/RobotHWSim</plugin>
+        </hardware>
+        <joint name="left_wheel_joint">
+            <command_interface name="velocity"/>
+            <state_interface name="position"/>
+            <state_interface name="velocity"/>
+        </joint>
+        <joint name="right_wheel_joint">
+            <command_interface name="velocity"/>
+            <state_interface name="position"/>
+            <state_interface name="velocity"/>
+        </joint>
+    </ros2_control>
 </robot>

File: tp1_robot/urdf/inertial_macros.xacro (robot description, xacro)
@@ -1,13 +1,12 @@
 <?xml version="1.0"?>
-<robot xmlns:xacro="http://www.ros.org/wiki/xacro" >
-    <!-- Specify some standard inertial calculations https://en.wikipedia.org/wiki/List_of_moments_of_inertia -->
-    <!-- These make use of xacro's mathematical functionality -->
+<robot xmlns:xacro="http://www.ros.org/wiki/xacro">
+    <!-- Macros de inercia -->
     <xacro:macro name="inertial_sphere" params="mass radius *origin">
         <inertial>
             <xacro:insert_block name="origin"/>
-            <mass value="${mass}" />
+            <mass value="${mass}"/>
             <inertia ixx="${(2/5) * mass * (radius*radius)}" ixy="0.0" ixz="0.0"
-                    iyy="${(2/5) * mass * (radius*radius)}" iyz="0.0"
-                    izz="${(2/5) * mass * (radius*radius)}" />
+                     iyy="${(2/5) * mass * (radius*radius)}" iyz="0.0"
+                     izz="${(2/5) * mass * (radius*radius)}"/>
         </inertial>
     </xacro:macro>
@@ -15,8 +14,8 @@
         <inertial>
             <xacro:insert_block name="origin"/>
-            <mass value="${mass}" />
-            <inertia ixx="${(1/12) * mass * (y*y+z*z)}" ixy="0.0" ixz="0.0"
-                    iyy="${(1/12) * mass * (x*x+z*z)}" iyz="0.0"
-                    izz="${(1/12) * mass * (x*x+y*y)}" />
+            <mass value="${mass}"/>
+            <inertia ixx="${(1/12) * mass * (y*y + z*z)}" ixy="0.0" ixz="0.0"
+                     iyy="${(1/12) * mass * (x*x + z*z)}" iyz="0.0"
+                     izz="${(1/12) * mass * (x*x + y*y)}"/>
         </inertial>
     </xacro:macro>
@@ -24,10 +23,11 @@
         <inertial>
             <xacro:insert_block name="origin"/>
-            <mass value="${mass}" />
+            <mass value="${mass}"/>
             <inertia ixx="${(1/12) * mass * (3*radius*radius + length*length)}" ixy="0.0" ixz="0.0"
-                    iyy="${(1/12) * mass * (3*radius*radius + length*length)}" iyz="0.0"
-                    izz="${(1/2) * mass * (radius*radius)}" />
+                     iyy="${(1/12) * mass * (3*radius*radius + length*length)}" iyz="0.0"
+                     izz="${(1/2) * mass * (radius*radius)}"/>
         </inertial>
     </xacro:macro>
+    <!-- Inercia dummy -->
     <xacro:macro name="dummy_inertial">
         <inertial>
@@ -39,28 +39,12 @@
         </inertial>
     </xacro:macro>
-    <!-- RVIZ material RGBA definition -->
-    <material name="red">
-        <color rgba="0.8 0.0 0.0 1.0"/>
-    </material>
-    <material name="green">
-        <color rgba="0.0 0.8 0.0 1.0"/>
-    </material>
-    <material name="blue">
-        <color rgba="0.0 0.0 0.8 1.0"/>
-    </material>
-    <material name="black">
-        <color rgba="0 0 0 1"/>
-    </material>
-    <material name="white">
-        <color rgba="1 1 1 1"/>
-    </material>
-    <material name="orange">
-        <color rgba="1 0.3 0.1 1"/>
-    </material>
-    <material name="silver">
-        <color rgba="0.79 0.82 0.93 1"/>
-    </material>
-    <material name="dark_grey">
-        <color rgba="0.3 0.3 0.3 1"/>
-    </material>
+    <!-- Materiales -->
+    <material name="red"><color rgba="0.8 0.0 0.0 1.0"/></material>
+    <material name="green"><color rgba="0.0 0.8 0.0 1.0"/></material>
+    <material name="blue"><color rgba="0.0 0.0 0.8 1.0"/></material>
+    <material name="black"><color rgba="0 0 0 1"/></material>
+    <material name="white"><color rgba="1 1 1 1"/></material>
+    <material name="orange"><color rgba="1 0.3 0.1 1"/></material>
+    <material name="silver"><color rgba="0.79 0.82 0.93 1"/></material>
+    <material name="dark_grey"><color rgba="0.3 0.3 0.3 1"/></material>
 </robot>

File: tp1_robot/urdf/motor.xacro (robot description, xacro)
@@ -1,5 +1,6 @@
 <?xml version="1.0"?>
-<robot xmlns:xacro="http://www.ros.org/wiki/xacro" >
+<robot xmlns:xacro="http://www.ros.org/wiki/xacro">
     <xacro:macro name="motor" params="prefix chassis_width:=0 reflect:=false">
+        <!-- Parámetros -->
         <xacro:property name="motor_mass" value="0.1"/>
         <xacro:property name="motor_x_size" value="0.07"/>
@@ -12,17 +13,20 @@
         <xacro:property name="pos_y_joint" value="${(chassis_width/2) - motor_y_offset + (motor_y_size/2)}"/>
         <xacro:property name="pos_z_joint" value="${motor_z_offset}"/>
+        <!-- Link del motor -->
         <link name="${prefix}_motor">
+            <!-- Visual -->
             <visual>
                 <origin xyz="0 0 0" rpy="0 0 0"/>
                 <geometry>
                     <xacro:if value="${reflect}">
-                        <mesh filename="file://$(find tp1_robot)/meshes/motor.stl" scale="1 -1 1" />
+                        <mesh filename="file://$(find tp1_robot)/meshes/motor.stl" scale="1 -1 1"/>
                     </xacro:if>
                     <xacro:unless value="${reflect}">
-                        <mesh filename="file://$(find tp1_robot)/meshes/motor.stl" />
+                        <mesh filename="file://$(find tp1_robot)/meshes/motor.stl"/>
                     </xacro:unless>
                 </geometry>
                 <material name="blue"/>
             </visual>
+            <!-- Colisión -->
             <collision>
                 <origin xyz="0 0 0" rpy="0 0 0"/>
@@ -31,13 +35,15 @@
                 </geometry>
             </collision>
+            <!-- Inercia -->
             <xacro:inertial_box mass="${motor_mass}" x="${motor_x_size}" y="${motor_y_size}" z="${motor_z_size}">
                 <origin xyz="0 0 0" rpy="0 0 0"/>
             </xacro:inertial_box>
         </link>
+        <!-- Joint del motor -->
         <joint name="${prefix}_motor_joint" type="fixed">
             <parent link="base_link"/>
             <child link="${prefix}_motor"/>
             <xacro:if value="${reflect}">
-                <origin xyz="${pos_x_joint} ${-pos_y_joint} ${pos_z_joint}" rpy="0 0 0"/>
+                <origin xyz="${pos_x_joint} ${-1 * pos_y_joint} ${pos_z_joint}" rpy="0 0 0"/>
             </xacro:if>
             <xacro:unless value="${reflect}">
@@ -45,4 +51,4 @@
             </xacro:unless>
         </joint>
-	</xacro:macro>
+    </xacro:macro>
 </robot>

Commit message: tp1_robot_V0.8

File: tp1_robot/urdf/diffbot.xacro (robot description, xacro)
@@ -2,127 +2,186 @@
 <robot name="diffbot" xmlns:xacro="http://www.ros.org/wiki/xacro">
   <!-- Propiedades -->
+  <!-- Masa del chasis en kilogramos -->
   <xacro:property name="chassis_mass" value="0.8"/>
+  <!-- Radio de cada rueda en metros -->
   <xacro:property name="wheel_radius" value="0.035"/>
+  <!-- Ancho (longitud del cilindro) de cada rueda -->
   <xacro:property name="wheel_width" value="0.025"/>
+  <!-- Separación entre las ruedas izquierda y derecha -->
   <xacro:property name="wheel_separation" value="0.16"/>
   <!-- Includes -->
+  <!-- Incluye macros para definir inercia -->
   <xacro:include filename="$(find tp1_robot)/urdf/inertial_macros.xacro"/>
+  <!-- Incluye definición del motor -->
   <xacro:include filename="$(find tp1_robot)/urdf/motor.xacro"/>
   <!-- Chasis -->
+  <!-- Enlace principal del robot (base) -->
   <link name="base_link">
     <visual>
+      <!-- Posición y orientación del mesh visual respecto al link (x,y,z / roll,pitch,yaw) -->
       <origin xyz="0 0 0" rpy="0 0 0"/>
       <geometry>
+        <!-- Malla 3D del chasis -->
         <mesh filename="file://$(find tp1_robot)/meshes/chassis.stl"/>
       </geometry>
     </visual>
     <collision>
+      <!-- Posición y orientación de la geometría de colisión -->
       <origin xyz="0 0 0" rpy="0 0 0"/>
       <geometry>
+        <!-- Caja de colisión con dimensiones en x,y,z -->
         <box size="0.195 0.1 0.05"/>
       </geometry>
     </collision>
+    <!-- Inercia del chasis, coincide con la caja de colisión -->
     <xacro:inertial_box mass="${chassis_mass}" x="0.195" y="0.1" z="0.05">
+    <!-- Centro de masa en el origen del link -->
       <origin xyz="0 0 0" rpy="0 0 0"/>
     </xacro:inertial_box>
   </link>
   <!-- Ruedas -->
+  <!-- Macro para definir una rueda -->
   <xacro:macro name="wheel" params="prefix xyz axis">
+    <!-- Nombre del link de la rueda (left/right) -->
     <link name="${prefix}_wheel">
       <visual>
+        <!-- Gira el cilindro 90° sobre el eje X para que se oriente correctamente -->
         <origin xyz="0 0 0" rpy="1.5708 0 0"/>
         <geometry>
+          <!-- Geometría cilíndrica de la rueda -->
           <cylinder radius="${wheel_radius}" length="${wheel_width}"/>
         </geometry>
       </visual>
       <collision>
+        <!-- Igual que visual, gira el cilindro sobre X -->
         <origin xyz="0 0 0" rpy="1.5708 0 0"/>
         <geometry>
+          <!-- Geometría de colisión de la rueda -->
           <cylinder radius="${wheel_radius}" length="${wheel_width}"/>
         </geometry>
       </collision>
     </link>
+    <!-- Unión continua entre base_link y la rueda -->
     <joint name="${prefix}_wheel_joint" type="continuous">
+      <!-- Posición de la rueda respecto a base_link (X adelante, Y lateral, Z altura) -->
       <origin xyz="${xyz}" rpy="0 0 0"/>
+      <!-- Elemento padre es el chasis -->
       <parent link="base_link"/>
+      <!-- Hijo es la rueda correspondiente -->
       <child link="${prefix}_wheel"/>
+      <!-- Eje de rotación de la rueda (0 1 0) indica giro sobre eje Y -->
       <axis xyz="${axis}"/>
     </joint>
   </xacro:macro>
   <!-- Instancias de ruedas -->
+  <!-- Rueda izquierda: un poco hacia adelante, desplazada a la izquierda y por debajo -->
   <xacro:wheel prefix="left"  xyz="0.0175  0.065 -0.0175" axis="0 1 0"/>
+  <!-- Rueda derecha: simétrica, desplazada a la derecha -->
   <xacro:wheel prefix="right" xyz="0.0175 -0.065 -0.0175" axis="0 1 0"/>
   <!-- Motores -->
+  <!-- Motor izquierdo, no reflejado -->
   <xacro:motor prefix="left" chassis_width="0.1" reflect="false"/>
+  <!-- Motor derecho, reflejado para simetría -->
   <xacro:motor prefix="right" chassis_width="0.1" reflect="true"/>
   <!-- Caster Base -->
+  <!-- Base del soporte trasero (caster) -->
   <link name="caster_base">
     <visual>
-      <origin xyz="0.08 0 0" rpy="0 0 0"/>
+      <!-- Adelantado respecto al link padre base_link -->
+      <origin xyz="0.0 0 0.0045" rpy="0 0 0"/>
       <geometry>
+        <!-- Malla visual del soporte base -->
         <mesh filename="file://$(find tp1_robot)/meshes/caster_base.stl"/>
       </geometry>
     </visual>
   </link>
+  <!-- Unión fija al chasis -->
   <joint name="caster_base_joint" type="fixed">
     <parent link="base_link"/>
     <child link="caster_base"/>
+    <!-- Posición respecto a base_link: adelante y más abajo -->
     <origin xyz="0.08 0 -0.025" rpy="0 0 0"/>
   </joint>
   <!-- Caster Wheel -->
+  <!-- Rueda trasera del caster -->
   <link name="caster_wheel">
     <visual>
-      <origin xyz="0 0 -0.01" rpy="0 0 0"/>
+      <!-- Debajo del caster_base -->
+      <origin xyz="-0.015 0 -0.020" rpy="0 0 0"/>
       <geometry>
+        <!-- Malla de la rueda libre trasera -->
         <mesh filename="file://$(find tp1_robot)/meshes/caster_wheel.stl"/>
       </geometry>
     </visual>
   </link>
+  <!-- Unión fija a caster_base -->
   <joint name="caster_wheel_joint" type="fixed">
     <parent link="caster_base"/>
     <child link="caster_wheel"/>
+    <!-- Posicionada justo debajo -->
     <origin xyz="0 0 -0.01" rpy="0 0 0"/>
   </joint>
   <!-- Caster Wheel Support -->
+  <!-- Soporte de la rueda trasera -->
   <link name="caster_wheel_support">
     <visual>
+      <!-- Coincide con caster_wheel -->
       <origin xyz="0 0 0" rpy="0 0 0"/>
       <geometry>
+        <!-- Malla del soporte -->
         <mesh filename="file://$(find tp1_robot)/meshes/caster_wheel_support.stl"/>
       </geometry>
     </visual>
   </link>
+  <!-- Unión fija a la rueda trasera -->
   <joint name="caster_support_joint" type="fixed">
     <parent link="caster_wheel"/>
     <child link="caster_wheel_support"/>
+    <!-- Mismo origen que la rueda trasera -->
     <origin xyz="0 0 0" rpy="0 0 0"/>
   </joint>
   <!-- Transformación odom -->
+  <!-- Enlace lógico para la odometría -->
   <link name="odom"/>
+  <!-- Unión entre el marco de odometría y la base -->
   <joint name="odom_to_base_link" type="fixed">
     <parent link="odom"/>
     <child link="base_link"/>
+    <!-- Sin transformación: los marcos coinciden -->
     <origin xyz="0 0 0" rpy="0 0 0"/>
   </joint>
   <!-- Plugin Gazebo -->
   <gazebo>
+    <!-- Plugin para control diferencial en Gazebo -->
     <plugin name="gazebo_ros_control" filename="libgazebo_ros_diff_drive.so">
+      <!-- Namespace para los tópicos -->
       <ros><namespace>/diffbot</namespace></ros>
+      <!-- Distancia entre ruedas -->
       <wheel_separation>${wheel_separation}</wheel_separation>
+      <!-- Diámetro de la rueda (2 * radio) -->
       <wheel_diameter>0.07</wheel_diameter>
+      <!-- Nombre del joint de la rueda izquierda -->
       <left_joint>left_wheel_joint</left_joint>
+      <!-- Nombre del joint de la rueda derecha -->
       <right_joint>right_wheel_joint</right_joint>
     </plugin>
   </gazebo>
   <!-- ROS2 Control -->
+  <!-- Controlador ROS2 para el robot -->
   <ros2_control name="diffbot_controller" type="system">
     <hardware>
+      <!-- Plugin de simulación para hardware -->
       <plugin>gazebo_ros2_control/RobotHWSim</plugin>
     </hardware>
+    <!-- Control sobre la rueda izquierda -->
     <joint name="left_wheel_joint">
+      <!-- Se puede enviar velocidad -->
       <command_interface name="velocity"/>
+      <!-- Se puede leer la posición -->
       <state_interface name="position"/>
+      <!-- Se puede leer la velocidad -->
       <state_interface name="velocity"/>
     </joint>
+    <!-- Igual que la izquierda pero para la rueda derecha -->
     <joint name="right_wheel_joint">
       <command_interface name="velocity"/>
