Commit message: tp1_robot_V0.11

File: tp1_robot/urdf/diffbot.xacro (robot description, xacro)
@@ -30,17 +30,17 @@
   <link name="base_link">
     <visual>
-      <origin xyz="0 0 0" rpy="0 0 0"/> <!-- Posición y orientación visual del chasis -->
+      <origin xyz="0 0 0" rpy="0 0 0"/>
       <geometry>
-        <mesh filename="file://$(find tp1_robot)/meshes/chassis.stl"/> <!-- Malla visual -->
+        <mesh filename="file://$(find tp1_robot)/meshes/chassis.stl"/>
       </geometry>
     </visual>
     <collision>
-      <origin xyz="0 0 0" rpy="0 0 0"/> <!-- Posición y orientación de colisiones -->
+      <origin xyz="0 0 0" rpy="0 0 0"/>
       <geometry>
-        <box size="0.195 0.1 0.05"/> <!-- Tamaño de la caja de colisión: largo, ancho, alto (m) -->
+        <box size="0.195 0.1 0.05"/>
       </geometry>
     </collision>
     <xacro:inertial_box mass="${chassis_mass}" x="0.195" y="0.1" z="0.05">
-      <origin xyz="0 0 0" rpy="0 0 0"/> <!-- Centro de masa -->
+      <origin xyz="0 0 0" rpy="0 0 0"/>
     </xacro:inertial_box>
   </link>
@@ -51,7 +51,7 @@
     <link name="${prefix}_wheel">
       <visual>
-        <origin xyz="0 0 0" rpy="1.5708 0 0"/> <!-- Rueda girada para estar vertical -->
+        <origin xyz="0 0 0" rpy="1.5708 0 0"/>
         <geometry>
-          <cylinder radius="${wheel_radius}" length="${wheel_width}"/> <!-- Cilindro como rueda -->
+          <cylinder radius="${wheel_radius}" length="${wheel_width}"/>
         </geometry>
         <material name="${wheel_color}"/>
@@ -66,8 +66,8 @@
     </link>
     <joint name="${prefix}_wheel_joint" type="continuous">
-      <origin xyz="${xyz}" rpy="0 0 0"/> <!-- Posición de la rueda respecto al chasis -->
+      <origin xyz="${xyz}" rpy="0 0 0"/>
       <parent link="base_link"/>
       <child link="${prefix}_wheel"/>
-      <axis xyz="${axis}"/> <!-- Eje de rotación de la rueda -->
+      <axis xyz="${axis}"/>
     </joint>
   </xacro:macro>
@@ -75,8 +75,8 @@
   <!-- === Ruedas izquierda y derecha === -->
   <!-- ======================= -->
-  <xacro:wheel prefix="left"  xyz="0.0175  0.065 -0.0175" axis="0 1 0"/> <!-- Rueda izquierda -->
-  <xacro:wheel prefix="right" xyz="0.0175 -0.065 -0.0175" axis="0 1 0"/> <!-- Rueda derecha -->
-  <xacro:motor prefix="left" chassis_width="0.1" reflect="false"/> <!-- Motor izquierdo -->
-  <xacro:motor prefix="right" chassis_width="0.1" reflect="true"/> <!-- Motor derecho -->
+  <xacro:wheel prefix="left" xyz="0.0175  0.065 -0.0175" axis="0 1 0"/>
+  <xacro:wheel prefix="right" xyz="0.0175 -0.065 -0.0175" axis="0 1 0"/>
+  <xacro:motor prefix="left" chassis_width="0.1" reflect="false"/>
+  <xacro:motor prefix="right" chassis_width="0.1" reflect="true"/>
   <!-- ======================= -->
   <!-- === Caster trasero (rueda loca) === -->
@@ -95,5 +95,5 @@
     <parent link="base_link"/>
     <child link="caster"/>
-    <origin xyz="${caster_origin_xyz}" rpy="0 0 0"/> <!-- Posición del caster respecto al chasis -->
+    <origin xyz="${caster_origin_xyz}" rpy="0 0 0"/>
   </joint>
   <!-- Rueda rotante del caster -->
@@ -110,6 +110,6 @@
     <parent link="caster"/>
     <child link="caster_wheel"/>
-    <origin xyz="0 0 -0.01" rpy="0 0 0"/> <!-- Eje de giro libre -->
-    <axis xyz="0 0 1"/> <!-- Rueda gira libremente en z -->
+    <origin xyz="0 0 -0.01" rpy="0 0 0"/>
+    <axis xyz="0 0 1"/>
   </joint>
   <!-- Soporte de la rueda del caster -->
@@ -126,31 +126,28 @@
     <parent link="caster_wheel"/>
     <child link="caster_wheel_support"/>
-    <origin xyz="0 0 0" rpy="0 0 0"/> <!-- Unido directamente sin movimiento -->
+    <origin xyz="0 0 0" rpy="0 0 0"/>
   </joint>
   <!-- ======================= -->
-  <!-- === Odometría del robot === -->
-  <!-- ======================= -->
-  <link name="odom"/>
-  <joint name="odom_to_base_link" type="fixed">
-    <parent link="odom"/>
-    <child link="base_link"/>
-    <origin xyz="0 0 0" rpy="0 0 0"/> <!-- Sistema de referencia absoluto -->
-  </joint>
-  <!-- ======================= -->
-  <!-- === Plugin de Gazebo para ROS1 === -->
+  <!-- === Plugin de Gazebo para ROS 2 === -->
   <!-- ======================= -->
   <gazebo>
-    <plugin name="gazebo_ros_control" filename="libgazebo_ros_diff_drive.so">
-      <ros><namespace>/diffbot</namespace></ros>
+    <plugin name="gazebo_ros_diff_drive" filename="libgazebo_ros_diff_drive.so">
+      <ros>
+        <namespace>/diffbot</namespace>
+      </ros>
       <wheel_separation>${wheel_separation}</wheel_separation>
       <wheel_diameter>0.07</wheel_diameter>
       <left_joint>left_wheel_joint</left_joint>
       <right_joint>right_wheel_joint</right_joint>
+      <publish_odom>true</publish_odom>
+      <publish_odom_tf>true</publish_odom_tf>
+      <update_rate>50</update_rate>
+      <torque>5.0</torque>
     </plugin>
   </gazebo>
   <!-- ======================= -->
-  <!-- === Controlador ROS 2 === -->
+  <!-- === ROS 2 Control === -->
   <!-- ======================= -->
-  <ros2_control name="diffbot_controller" type="system">
+  <ros2_control name="diffbot_ros2_control" type="system">
     <hardware>
       <plugin>gazebo_ros2_control/RobotHWSim</plugin>

File: tp1_robot/urdf/inertial_macros.xacro (robot description, xacro)
@@ -1,50 +1,92 @@
 <?xml version="1.0"?>
 <robot xmlns:xacro="http://www.ros.org/wiki/xacro">
-    <!-- Macros de inercia -->
-    <xacro:macro name="inertial_sphere" params="mass radius *origin">
-        <inertial>
-            <xacro:insert_block name="origin"/>
-            <mass value="${mass}"/>
-            <inertia ixx="${(2/5) * mass * (radius*radius)}" ixy="0.0" ixz="0.0"
-                     iyy="${(2/5) * mass * (radius*radius)}" iyz="0.0"
-                     izz="${(2/5) * mass * (radius*radius)}"/>
-        </inertial>
-    </xacro:macro>
-    <xacro:macro name="inertial_box" params="mass x y z *origin">
-        <inertial>
-            <xacro:insert_block name="origin"/>
-            <mass value="${mass}"/>
-            <inertia ixx="${(1/12) * mass * (y*y + z*z)}" ixy="0.0" ixz="0.0"
-                     iyy="${(1/12) * mass * (x*x + z*z)}" iyz="0.0"
-                     izz="${(1/12) * mass * (x*x + y*y)}"/>
-        </inertial>
-    </xacro:macro>
-    <xacro:macro name="inertial_cylinder" params="mass length radius *origin">
-        <inertial>
-            <xacro:insert_block name="origin"/>
-            <mass value="${mass}"/>
-            <inertia ixx="${(1/12) * mass * (3*radius*radius + length*length)}" ixy="0.0" ixz="0.0"
-                     iyy="${(1/12) * mass * (3*radius*radius + length*length)}" iyz="0.0"
-                     izz="${(1/2) * mass * (radius*radius)}"/>
-        </inertial>
-    </xacro:macro>
-    <!-- Inercia dummy -->
-    <xacro:macro name="dummy_inertial">
-        <inertial>
-            <origin xyz="0 0 0" rpy="0 0 0"/>
-            <mass value="0.001"/>
-            <inertia ixx="0.00001" ixy="0" ixz="0"
-                     iyy="0.00001" iyz="0"
-                     izz="0.00001"/>
-        </inertial>
-    </xacro:macro>
-    <!-- Materiales -->
-    <material name="red"><color rgba="0.8 0.0 0.0 1.0"/></material>
-    <material name="green"><color rgba="0.0 0.8 0.0 1.0"/></material>
-    <material name="blue"><color rgba="0.0 0.0 0.8 1.0"/></material>
-    <material name="black"><color rgba="0 0 0 1"/></material>
-    <material name="white"><color rgba="1 1 1 1"/></material>
-    <material name="orange"><color rgba="1 0.3 0.1 1"/></material>
-    <material name="silver"><color rgba="0.79 0.82 0.93 1"/></material>
-    <material name="dark_grey"><color rgba="0.3 0.3 0.3 1"/></material>
+  <!-- ======================= -->
+  <!-- === Macros de Inercia === -->
+  <!-- ======================= -->
+  <!-- Macro para inercia de esfera -->
+  <!-- Parámetros:
+       - mass: Masa del objeto (kg)
+       - radius: Radio de la esfera (m)
+       - origin: Origen del centro de masa -->
+  <xacro:macro name="inertial_sphere" params="mass radius *origin">
+    <inertial>
+      <xacro:insert_block name="origin"/>
+      <mass value="${mass}"/>
+      <inertia ixx="${(2/5) * mass * (radius*radius)}" ixy="0.0" ixz="0.0"
+               iyy="${(2/5) * mass * (radius*radius)}" iyz="0.0"
+               izz="${(2/5) * mass * (radius*radius)}"/>
+    </inertial>
+  </xacro:macro>
+  <!-- Macro para inercia de caja -->
+  <!-- Parámetros:
+       - mass: Masa del objeto (kg)
+       - x, y, z: Dimensiones de la caja (m)
+       - origin: Origen del centro de masa -->
+  <xacro:macro name="inertial_box" params="mass x y z *origin">
+    <inertial>
+      <xacro:insert_block name="origin"/>
+      <mass value="${mass}"/>
+      <inertia ixx="${(1/12) * mass * (y*y + z*z)}" ixy="0.0" ixz="0.0"
+               iyy="${(1/12) * mass * (x*x + z*z)}" iyz="0.0"
+               izz="${(1/12) * mass * (x*x + y*y)}"/>
+    </inertial>
+  </xacro:macro>
+  <!-- Macro para inercia de cilindro -->
+  <!-- Parámetros:
+       - mass: Masa del objeto (kg)
+       - length: Longitud del cilindro (m)
+       - radius: Radio del cilindro (m)
+       - origin: Origen del centro de masa -->
+  <xacro:macro name="inertial_cylinder" params="mass length radius *origin">
+    <inertial>
+      <xacro:insert_block name="origin"/>
+      <mass value="${mass}"/>
+      <inertia ixx="${(1/12) * mass * (3*radius*radius + length*length)}" ixy="0.0" ixz="0.0"
+               iyy="${(1/12) * mass * (3*radius*radius + length*length)}" iyz="0.0"
+               izz="${(1/2) * mass * (radius*radius)}"/>
+    </inertial>
+  </xacro:macro>
+  <!-- Macro de inercia dummy (para links sin masa real) -->
+  <!-- Ejemplo: sensores o estructuras ligeras -->
+  <xacro:macro name="dummy_inertial">
+    <inertial>
+      <origin xyz="0 0 0" rpy="0 0 0"/>
+      <mass value="0.001"/>
+      <inertia ixx="0.00001" ixy="0" ixz="0"
+               iyy="0.00001" iyz="0"
+               izz="0.00001"/>
+    </inertial>
+  </xacro:macro>
+  <!-- ======================= -->
+  <!-- === Materiales === -->
+  <!-- ======================= -->
+  <!-- Colores estándar -->
+  <material name="red">
+    <color rgba="0.8 0.0 0.0 1.0"/>
+  </material>
+  <material name="green">
+    <color rgba="0.0 0.8 0.0 1.0"/>
+  </material>
+  <material name="blue">
+    <color rgba="0.0 0.0 0.8 1.0"/>
+  </material>
+  <material name="black">
+    <color rgba="0 0 0 1"/>
+  </material>
+  <material name="white">
+    <color rgba="1 1 1 1"/>
+  </material>
+  <material name="orange">
+    <color rgba="1 0.3 0.1 1"/>
+  </material>
+  <material name="silver">
+    <color rgba="0.79 0.82 0.93 1"/>
+  </material>
+  <material name="dark_grey">
+    <color rgba="0.3 0.3 0.3 1"/>
+  </material>
+  <!-- Color adicional para ruedas -->
+  <material name="wheel_color">
+    <color rgba="0.6 0.6 0.6 1"/>
+  </material>
 </robot>

File: tp1_robot/urdf/motor.xacro (robot description, xacro)
@@ -1,54 +1,73 @@
 <?xml version="1.0"?>
 <robot xmlns:xacro="http://www.ros.org/wiki/xacro">
-    <xacro:macro name="motor" params="prefix chassis_width:=0 reflect:=false">
-        <!-- Parámetros -->
-        <xacro:property name="motor_mass" value="0.1"/>
-        <xacro:property name="motor_x_size" value="0.07"/>
-        <xacro:property name="motor_y_size" value="0.0188"/>
-        <xacro:property name="motor_z_size" value="0.0225"/>
-        <xacro:property name="motor_x_offset" value="0.0015"/>
-        <xacro:property name="motor_y_offset" value="0.0216"/>
-        <xacro:property name="motor_z_offset" value="-0.017"/>
-        <xacro:property name="pos_x_joint" value="${motor_x_offset}"/>
-        <xacro:property name="pos_y_joint" value="${(chassis_width/2) - motor_y_offset + (motor_y_size/2)}"/>
-        <xacro:property name="pos_z_joint" value="${motor_z_offset}"/>
-        <!-- Link del motor -->
-        <link name="${prefix}_motor">
-            <!-- Visual -->
-            <visual>
-                <origin xyz="0 0 0" rpy="0 0 0"/>
-                <geometry>
-                    <xacro:if value="${reflect}">
-                        <mesh filename="file://$(find tp1_robot)/meshes/motor.stl" scale="1 -1 1"/>
-                    </xacro:if>
-                    <xacro:unless value="${reflect}">
-                        <mesh filename="file://$(find tp1_robot)/meshes/motor.stl"/>
-                    </xacro:unless>
-                </geometry>
-                <material name="blue"/>
-            </visual>
-            <!-- Colisión -->
-            <collision>
-                <origin xyz="0 0 0" rpy="0 0 0"/>
-                <geometry>
-                    <box size="${motor_x_size} ${motor_y_size} ${motor_z_size}"/>
-                </geometry>
-            </collision>
-            <!-- Inercia -->
-            <xacro:inertial_box mass="${motor_mass}" x="${motor_x_size}" y="${motor_y_size}" z="${motor_z_size}">
-                <origin xyz="0 0 0" rpy="0 0 0"/>
-            </xacro:inertial_box>
-        </link>
-        <!-- Joint del motor -->
-        <joint name="${prefix}_motor_joint" type="fixed">
-            <parent link="base_link"/>
-            <child link="${prefix}_motor"/>
-            <xacro:if value="${reflect}">
-                <origin xyz="${pos_x_joint} ${-1 * pos_y_joint} ${pos_z_joint}" rpy="0 0 0"/>
-            </xacro:if>
-            <xacro:unless value="${reflect}">
-                <origin xyz="${pos_x_joint} ${pos_y_joint} ${pos_z_joint}" rpy="0 0 0"/>
-            </xacro:unless>
-        </joint>
-    </xacro:macro>
+  <!-- ======================= -->
+  <!-- === Macro de Motor === -->
+  <!-- ======================= -->
+  <!-- Este macro inserta un motor en el chasis del robot.
+       Se puede usar para ambos lados (izquierdo o derecho)
+       Parametrizado para posicionar correctamente el motor según el ancho del chasis.
+       Opcionalmente se puede reflejar para el lado derecho. -->
+  <!-- === Parámetros del macro === -->
+  <!-- prefix: prefijo para los nombres del link y joint (ej: left, right) -->
+  <!-- chassis_width: ancho total del chasis (usado para calcular posición Y del motor) -->
+  <!-- reflect: booleano que indica si el motor debe ser reflejado (para el lado derecho) -->
+  <xacro:macro name="motor" params="prefix chassis_width:=0 reflect:=false">
+    <!-- === Propiedades físicas del motor === -->
+    <!-- Masa del motor en kilogramos -->
+    <xacro:property name="motor_mass" value="0.1"/>
+    <!-- Dimensiones del motor en metros (x, y, z) -->
+    <xacro:property name="motor_x_size" value="0.07"/>
+    <xacro:property name="motor_y_size" value="0.0188"/>
+    <xacro:property name="motor_z_size" value="0.0225"/>
+    <!-- Desplazamiento del motor respecto al centro del chasis -->
+    <xacro:property name="motor_x_offset" value="0.0015"/>
+    <xacro:property name="motor_y_offset" value="0.0216"/>
+    <xacro:property name="motor_z_offset" value="-0.017"/>
+    <!-- Cálculo automático de posición Y del joint -->
+    <xacro:property name="pos_y_joint"
+      value="${(chassis_width / 2) - motor_y_offset + (motor_y_size / 2)}"/>
+    <!-- Posición fija del joint en X y Z -->
+    <xacro:property name="pos_x_joint" value="${motor_x_offset}"/>
+    <xacro:property name="pos_z_joint" value="${motor_z_offset}"/>
+    <!-- === Definición del link del motor === -->
+    <link name="${prefix}_motor">
+      <!-- === Visualización del motor === -->
+      <visual>
+        <origin xyz="0 0 0" rpy="0 0 0"/>
+        <geometry>
+          <!-- Si 'reflect' es true, escala negativo en Y para invertir orientación -->
+          <xacro:if value="${reflect}">
+            <mesh filename="file://$(find tp1_robot)/meshes/motor.stl" scale="1 -1 1"/>
+          </xacro:if>
+          <xacro:unless value="${reflect}">
+            <mesh filename="file://$(find tp1_robot)/meshes/motor.stl"/>
+          </xacro:unless>
+        </geometry>
+        <material name="blue"/>
+      </visual>
+      <!-- === Colisión del motor (caja simple para simuladores) === -->
+      <collision>
+        <origin xyz="0 0 0" rpy="0 0 0"/>
+        <geometry>
+          <box size="${motor_x_size} ${motor_y_size} ${motor_z_size}"/>
+        </geometry>
+      </collision>
+      <!-- === Inercia del motor (calculada automáticamente) === -->
+      <xacro:inertial_box mass="${motor_mass}" x="${motor_x_size}" y="${motor_y_size}" z="${motor_z_size}">
+        <origin xyz="0 0 0" rpy="0 0 0"/>
+      </xacro:inertial_box>
+    </link>
+    <!-- === Joint fijo entre el chasis y el motor === -->
+    <joint name="${prefix}_motor_joint" type="fixed">
+      <parent link="base_link"/>
+      <child link="${prefix}_motor"/>
+      <!-- Posicionamiento dinámico del motor -->
+      <xacro:if value="${reflect}">
+        <origin xyz="${pos_x_joint} ${-1 * pos_y_joint} ${pos_z_joint}" rpy="0 0 0"/>
+      </xacro:if>
+      <xacro:unless value="${reflect}">
+        <origin xyz="${pos_x_joint} ${pos_y_joint} ${pos_z_joint}" rpy="0 0 0"/>
+      </xacro:unless>
+    </joint>
+  </xacro:macro>
 </robot>

Commit message: tp1_robot_V0.12

File: tp1_robot/urdf/diffbot.xacro (robot description, xacro)
@@ -15,5 +15,5 @@
   <xacro:property name="wheel_color" value="silver"/>
   <!-- Posición del caster con respecto al centro del robot (x, y, z) en metros -->
-  <xacro:property name="caster_origin_xyz" value="-0.075 0 0.002"/>
+  <xacro:property name="caster_origin_xyz" value="-0.075 0 -0.007"/>
   <!-- Color del caster y sus partes -->
   <xacro:property name="caster_color" value="orange"/>
@@ -51,7 +51,7 @@
     <link name="${prefix}_wheel">
       <visual>
-        <origin xyz="0 0 0" rpy="1.5708 0 0"/>
+        <origin xyz="0 0 0" rpy="1.5708 0 0"/> <!-- Rotación base -->
         <geometry>
-          <cylinder radius="${wheel_radius}" length="${wheel_width}"/>
+          <mesh filename="file://$(find tp1_robot)/meshes/wheel.stl"/>
         </geometry>
         <material name="${wheel_color}"/>
@@ -60,13 +60,12 @@
         <origin xyz="0 0 0" rpy="1.5708 0 0"/>
         <geometry>
-          <cylinder radius="${wheel_radius}" length="${wheel_width}"/>
+          <mesh filename="file://$(find tp1_robot)/meshes/wheel.stl"/>
         </geometry>
-        <material name="${wheel_color}"/>
       </collision>
     </link>
     <joint name="${prefix}_wheel_joint" type="continuous">
-      <origin xyz="${xyz}" rpy="0 0 0"/>
       <parent link="base_link"/>
       <child link="${prefix}_wheel"/>
+      <origin xyz="${xyz}" rpy="0 0 0"/>
       <axis xyz="${axis}"/>
     </joint>
@@ -75,6 +74,35 @@
   <!-- === Ruedas izquierda y derecha === -->
   <!-- ======================= -->
-  <xacro:wheel prefix="left" xyz="0.0175  0.065 -0.0175" axis="0 1 0"/>
-  <xacro:wheel prefix="right" xyz="0.0175 -0.065 -0.0175" axis="0 1 0"/>
+  <!-- Rueda izquierda -->
+  <xacro:wheel prefix="left"
+               xyz="0.018  0.050 -0.018"
+               axis="0 1 0"/>
+  <!-- Rueda derecha con rotación extra de 180° en eje Z -->
+  <xacro:macro name="right_wheel_with_rotation">
+    <link name="right_wheel">
+      <visual>
+        <origin xyz="0 0 0" rpy="1.5708 0 3.1416"/> <!-- Rotación base + 180° extra en Z -->
+        <geometry>
+          <mesh filename="file://$(find tp1_robot)/meshes/wheel.stl"/>
+        </geometry>
+        <material name="${wheel_color}"/>
+      </visual>
+      <collision>
+        <origin xyz="0 0 0" rpy="1.5708 0 3.1416"/>
+        <geometry>
+          <mesh filename="file://$(find tp1_robot)/meshes/wheel.stl"/>
+        </geometry>
+      </collision>
+    </link>
+    <joint name="right_wheel_joint" type="continuous">
+      <parent link="base_link"/>
+      <child link="right_wheel"/>
+      <origin xyz="0.018 -0.050 -0.018" rpy="0 0 0"/>
+      <axis xyz="0 1 0"/>
+    </joint>
+  </xacro:macro>
+  <!-- Llamada a macro personalizada para rueda derecha rotada -->
+  <xacro:right_wheel_with_rotation/>
+  <!-- Motores -->
   <xacro:motor prefix="left" chassis_width="0.1" reflect="false"/>
   <xacro:motor prefix="right" chassis_width="0.1" reflect="true"/>
@@ -133,7 +161,5 @@
   <gazebo>
     <plugin name="gazebo_ros_diff_drive" filename="libgazebo_ros_diff_drive.so">
-      <ros>
-        <namespace>/diffbot</namespace>
-      </ros>
+      <ros><namespace>/diffbot</namespace></ros>
       <wheel_separation>${wheel_separation}</wheel_separation>
       <wheel_diameter>0.07</wheel_diameter>
