Commit message: tp1_robot_V0.13

File: tp1_robot/urdf/diffbot.xacro (robot description, xacro)
@@ -1,196 +1,101 @@
 <?xml version="1.0"?>
-<robot name="diffbot" xmlns:xacro="http://www.ros.org/wiki/xacro">
-  <!-- ======================= -->
-  <!-- === Propiedades === -->
-  <!-- ======================= -->
-  <!-- Masa del chasis en kilogramos -->
-  <xacro:property name="chassis_mass" value="0.8"/>
-  <!-- Radio de las ruedas (m) -->
-  <xacro:property name="wheel_radius" value="0.035"/>
-  <!-- Ancho de las ruedas (m) -->
-  <xacro:property name="wheel_width" value="0.025"/>
-  <!-- Separación entre las dos ruedas principales (m) -->
-  <xacro:property name="wheel_separation" value="0.16"/>
-  <!-- Color de las ruedas -->
-  <xacro:property name="wheel_color" value="silver"/>
-  <!-- Posición del caster con respecto al centro del robot (x, y, z) en metros -->
-  <xacro:property name="caster_origin_xyz" value="-0.075 0 -0.007"/>
-  <!-- Color del caster y sus partes -->
-  <xacro:property name="caster_color" value="orange"/>
-  <!-- ======================= -->
-  <!-- === Includes === -->
-  <!-- ======================= -->
-  <!-- Inclusión de macros para cálculo de masa -->
+<robot xmlns:xacro="http://ros.org/wiki/xacro"
+       xmlns:gazebo="http://www.gazebosim.org/schema/gazebo_urdf"
+       name="diffbot">
+  <!-- Parámetros reutilizables -->
+  <xacro:property name="PI" value="3.1415926535897931"/>
+  <xacro:property name="wheel_radius" value="0.035"/> <!-- Radio de rueda (m) -->
+  <xacro:property name="wheel_separation" value="0.23"/> <!-- Separación entre ruedas (m) -->
+  <!-- Incluir macros -->
   <xacro:include filename="$(find tp1_robot)/urdf/inertial_macros.xacro"/>
-  <!-- Inclusión de componentes para motores -->
   <xacro:include filename="$(find tp1_robot)/urdf/motor.xacro"/>
-  <!-- ======================= -->
-  <!-- === Chasis del robot === -->
-  <!-- ======================= -->
+  <!-- Base link (chasis) -->
   <link name="base_link">
     <visual>
-      <origin xyz="0 0 0" rpy="0 0 0"/>
       <geometry>
-        <mesh filename="file://$(find tp1_robot)/meshes/chassis.stl"/>
+        <mesh filename="package://tp1_robot/meshes/chassis.stl"/>
       </geometry>
+      <material name="gray"/>
     </visual>
     <collision>
-      <origin xyz="0 0 0" rpy="0 0 0"/>
       <geometry>
-        <box size="0.195 0.1 0.05"/>
+        <mesh filename="package://tp1_robot/meshes/chassis.stl"/>
       </geometry>
     </collision>
-    <xacro:inertial_box mass="${chassis_mass}" x="0.195" y="0.1" z="0.05">
-      <origin xyz="0 0 0" rpy="0 0 0"/>
-    </xacro:inertial_box>
+    <xacro:cylinder_inertia m="0.8" r="0.1" h="0.05"/>
   </link>
-  <!-- ======================= -->
-  <!-- === Macro para ruedas === -->
-  <!-- ======================= -->
-  <xacro:macro name="wheel" params="prefix xyz axis">
-    <link name="${prefix}_wheel">
-      <visual>
-        <origin xyz="0 0 0" rpy="1.5708 0 0"/> <!-- Rotación base -->
-        <geometry>
-          <mesh filename="file://$(find tp1_robot)/meshes/wheel.stl"/>
-        </geometry>
-        <material name="${wheel_color}"/>
-      </visual>
-      <collision>
-        <origin xyz="0 0 0" rpy="1.5708 0 0"/>
-        <geometry>
-          <mesh filename="file://$(find tp1_robot)/meshes/wheel.stl"/>
-        </geometry>
-      </collision>
-    </link>
-    <joint name="${prefix}_wheel_joint" type="continuous">
-      <parent link="base_link"/>
-      <child link="${prefix}_wheel"/>
-      <origin xyz="${xyz}" rpy="0 0 0"/>
-      <axis xyz="${axis}"/>
-    </joint>
-  </xacro:macro>
-  <!-- ======================= -->
-  <!-- === Ruedas izquierda y derecha === -->
-  <!-- ======================= -->
+  <!-- Ruedas -->
   <!-- Rueda izquierda -->
-  <xacro:wheel prefix="left"
-               xyz="0.018  0.050 -0.018"
-               axis="0 1 0"/>
-  <!-- Rueda derecha con rotación extra de 180° en eje Z -->
-  <xacro:macro name="right_wheel_with_rotation">
-    <link name="right_wheel">
-      <visual>
-        <origin xyz="0 0 0" rpy="1.5708 0 3.1416"/> <!-- Rotación base + 180° extra en Z -->
-        <geometry>
-          <mesh filename="file://$(find tp1_robot)/meshes/wheel.stl"/>
-        </geometry>
-        <material name="${wheel_color}"/>
-      </visual>
-      <collision>
-        <origin xyz="0 0 0" rpy="1.5708 0 3.1416"/>
-        <geometry>
-          <mesh filename="file://$(find tp1_robot)/meshes/wheel.stl"/>
-        </geometry>
-      </collision>
-    </link>
-    <joint name="right_wheel_joint" type="continuous">
-      <parent link="base_link"/>
-      <child link="right_wheel"/>
-      <origin xyz="0.018 -0.050 -0.018" rpy="0 0 0"/>
-      <axis xyz="0 1 0"/>
-    </joint>
-  </xacro:macro>
-  <!-- Llamada a macro personalizada para rueda derecha rotada -->
-  <xacro:right_wheel_with_rotation/>
-  <!-- Motores -->
+  <joint name="left_wheel_joint" type="continuous">
+    <parent link="base_link"/>
+    <child link="left_wheel_link"/>
+    <axis xyz="0 1 0"/>
+    <origin xyz="${-wheel_separation/2} -0.08 -0.035" rpy="0 0 0"/>
+  </joint>
+  <link name="left_wheel_link">
+    <visual>
+      <geometry>
+        <mesh filename="package://tp1_robot/meshes/wheel.stl"/>
+      </geometry>
+      <material name="black"/>
+    </visual>
+    <collision>
+      <geometry>
+        <mesh filename="package://tp1_robot/meshes/wheel.stl"/>
+      </geometry>
+    </collision>
+    <xacro:cylinder_inertia m="0.15" r="0.035" h="0.025"/>
+  </link>
+  <!-- Rueda derecha -->
+  <joint name="right_wheel_joint" type="continuous">
+    <parent link="base_link"/>
+    <child link="right_wheel_link"/>
+    <axis xyz="0 1 0"/>
+    <origin xyz="${wheel_separation/2} -0.08 -0.035" rpy="0 0 0"/>
+  </joint>
+  <link name="right_wheel_link">
+    <visual>
+      <geometry>
+        <mesh filename="package://tp1_robot/meshes/wheel.stl"/>
+      </geometry>
+      <material name="black"/>
+    </visual>
+    <collision>
+      <geometry>
+        <mesh filename="package://tp1_robot/meshes/wheel.stl"/>
+      </geometry>
+    </collision>
+    <xacro:cylinder_inertia m="0.15" r="0.035" h="0.025"/>
+  </link>
+  <!-- Motores (usando macro) -->
   <xacro:motor prefix="left" chassis_width="0.1" reflect="false"/>
   <xacro:motor prefix="right" chassis_width="0.1" reflect="true"/>
-  <!-- ======================= -->
-  <!-- === Caster trasero (rueda loca) === -->
-  <!-- ======================= -->
-  <!-- Base del caster -->
-  <link name="caster">
-    <visual>
-      <origin xyz="0 0 0.0045" rpy="0 0 0"/>
-      <geometry>
-        <mesh filename="file://$(find tp1_robot)/meshes/caster_base.stl"/>
-      </geometry>
-      <material name="${caster_color}"/>
-    </visual>
-  </link>
-  <joint name="caster_joint" type="fixed">
-    <parent link="base_link"/>
-    <child link="caster"/>
-    <origin xyz="${caster_origin_xyz}" rpy="0 0 0"/>
-  </joint>
-  <!-- Rueda rotante del caster -->
-  <link name="caster_wheel">
-    <visual>
-      <origin xyz="-0.015 0 -0.020" rpy="0 0 0"/>
-      <geometry>
-        <mesh filename="file://$(find tp1_robot)/meshes/caster_wheel.stl"/>
-      </geometry>
-      <material name="${caster_color}"/>
-    </visual>
-  </link>
-  <joint name="caster_wheel_joint" type="continuous">
-    <parent link="caster"/>
-    <child link="caster_wheel"/>
-    <origin xyz="0 0 -0.01" rpy="0 0 0"/>
-    <axis xyz="0 0 1"/>
-  </joint>
-  <!-- Soporte de la rueda del caster -->
-  <link name="caster_wheel_support">
-    <visual>
-      <origin xyz="0 0 0" rpy="0 0 0"/>
-      <geometry>
-        <mesh filename="file://$(find tp1_robot)/meshes/caster_wheel_support.stl"/>
-      </geometry>
-      <material name="${caster_color}"/>
-    </visual>
-  </link>
-  <joint name="caster_support_joint" type="fixed">
-    <parent link="caster_wheel"/>
-    <child link="caster_wheel_support"/>
-    <origin xyz="0 0 0" rpy="0 0 0"/>
-  </joint>
-  <!-- ======================= -->
-  <!-- === Plugin de Gazebo para ROS 2 === -->
-  <!-- ======================= -->
+  <!-- ROS2 Control -->
+  <ros2_control name="diffbot_ros2_control" type="system">
+    <hardware>
+      <plugin>gazebo_ros2_control/GazeboSystem</plugin>
+    </hardware>
+    <joint name="left_wheel_joint">
+      <command_interface name="velocity">
+        <param name="min">-10.0</param>
+        <param name="max">10.0</param>
+      </command_interface>
+      <state_interface name="velocity"/>
+      <state_interface name="position"/>
+    </joint>
+    <joint name="right_wheel_joint">
+      <command_interface name="velocity">
+        <param name="min">-10.0</param>
+        <param name="max">10.0</param>
+      </command_interface>
+      <state_interface name="velocity"/>
+      <state_interface name="position"/>
+    </joint>
+  </ros2_control>
+  <!-- Plugin para Gazebo -->
   <gazebo>
-    <plugin name="gazebo_ros_diff_drive" filename="libgazebo_ros_diff_drive.so">
-      <ros><namespace>/diffbot</namespace></ros>
-      <wheel_separation>${wheel_separation}</wheel_separation>
-      <wheel_diameter>0.07</wheel_diameter>
-      <left_joint>left_wheel_joint</left_joint>
-      <right_joint>right_wheel_joint</right_joint>
-      <publish_odom>true</publish_odom>
-      <publish_odom_tf>true</publish_odom_tf>
-      <update_rate>50</update_rate>
-      <torque>5.0</torque>
+    <plugin filename="libgazebo_ros2_control.so" name="gazebo_ros2_control">
+      <parameters>$(find tp1_robot)/config/diffbot_controllers.yaml</parameters>
     </plugin>
   </gazebo>
-  <!-- ======================= -->
-  <!-- === ROS 2 Control === -->
-  <!-- ======================= -->
-  <ros2_control name="diffbot_ros2_control" type="system">
-    <hardware>
-      <plugin>gazebo_ros2_control/RobotHWSim</plugin>
-    </hardware>
-    <joint name="left_wheel_joint">
-      <command_interface name="velocity"/>
-      <state_interface name="position"/>
-      <state_interface name="velocity"/>
-    </joint>
-    <joint name="right_wheel_joint">
-      <command_interface name="velocity"/>
-      <state_interface name="position"/>
-      <state_interface name="velocity"/>
-    </joint>
-    <joint name="caster_wheel_joint">
-      <state_interface name="position"/>
-      <state_interface name="velocity"/>
-    </joint>
-  </ros2_control>
 </robot>

File: tp1_robot/urdf/inertial_macros.xacro (robot description, xacro)
@@ -1,92 +1,30 @@
 <?xml version="1.0"?>
-<robot xmlns:xacro="http://www.ros.org/wiki/xacro">
-  <!-- ======================= -->
-  <!-- === Macros de Inercia === -->
-  <!-- ======================= -->
-  <!-- Macro para inercia de esfera -->
-  <!-- Parámetros:
-       - mass: Masa del objeto (kg)
-       - radius: Radio de la esfera (m)
-       - origin: Origen del centro de masa -->
-  <xacro:macro name="inertial_sphere" params="mass radius *origin">
+<robot xmlns:xacro="http://ros.org/wiki/xacro"
+       xmlns:gazebo="http://www.gazebosim.org/schema/gazebo_urdf">
+  <!-- Macro para inercia de un cilindro -->
+  <xacro:macro name="cylinder_inertia" params="m r h">
     <inertial>
-      <xacro:insert_block name="origin"/>
-      <mass value="${mass}"/>
-      <inertia ixx="${(2/5) * mass * (radius*radius)}" ixy="0.0" ixz="0.0"
-               iyy="${(2/5) * mass * (radius*radius)}" iyz="0.0"
-               izz="${(2/5) * mass * (radius*radius)}"/>
+      <mass value="${m}" />
+      <inertia
+        ixx="${m*(3*r*r + h*h)/12}"
+        ixy="0.0"
+        ixz="0.0"
+        iyy="${m*(3*r*r + h*h)/12}"
+        iyz="0.0"
+        izz="${m*r*r/2}" />
     </inertial>
   </xacro:macro>
-  <!-- Macro para inercia de caja -->
-  <!-- Parámetros:
-       - mass: Masa del objeto (kg)
-       - x, y, z: Dimensiones de la caja (m)
-       - origin: Origen del centro de masa -->
-  <xacro:macro name="inertial_box" params="mass x y z *origin">
+  <!-- Macro para inercia de un cubo -->
+  <xacro:macro name="box_inertia" params="m x y z">
     <inertial>
-      <xacro:insert_block name="origin"/>
-      <mass value="${mass}"/>
-      <inertia ixx="${(1/12) * mass * (y*y + z*z)}" ixy="0.0" ixz="0.0"
-               iyy="${(1/12) * mass * (x*x + z*z)}" iyz="0.0"
-               izz="${(1/12) * mass * (x*x + y*y)}"/>
+      <mass value="${m}" />
+      <inertia
+        ixx="${m*(y*y + z*z)/6}"
+        ixy="0.0"
+        ixz="0.0"
+        iyy="${m*(x*x + z*z)/6}"
+        iyz="0.0"
+        izz="${m*(x*x + y*y)/6}" />
     </inertial>
   </xacro:macro>
-  <!-- Macro para inercia de cilindro -->
-  <!-- Parámetros:
-       - mass: Masa del objeto (kg)
-       - length: Longitud del cilindro (m)
-       - radius: Radio del cilindro (m)
-       - origin: Origen del centro de masa -->
-  <xacro:macro name="inertial_cylinder" params="mass length radius *origin">
-    <inertial>
-      <xacro:insert_block name="origin"/>
-      <mass value="${mass}"/>
-      <inertia ixx="${(1/12) * mass * (3*radius*radius + length*length)}" ixy="0.0" ixz="0.0"
-               iyy="${(1/12) * mass * (3*radius*radius + length*length)}" iyz="0.0"
-               izz="${(1/2) * mass * (radius*radius)}"/>
-    </inertial>
-  </xacro:macro>
-  <!-- Macro de inercia dummy (para links sin masa real) -->
-  <!-- Ejemplo: sensores o estructuras ligeras -->
-  <xacro:macro name="dummy_inertial">
-    <inertial>
-      <origin xyz="0 0 0" rpy="0 0 0"/>
-      <mass value="0.001"/>
-      <inertia ixx="0.00001" ixy="0" ixz="0"
-               iyy="0.00001" iyz="0"
-               izz="0.00001"/>
-    </inertial>
-  </xacro:macro>
-  <!-- ======================= -->
-  <!-- === Materiales === -->
-  <!-- ======================= -->
-  <!-- Colores estándar -->
-  <material name="red">
-    <color rgba="0.8 0.0 0.0 1.0"/>
-  </material>
-  <material name="green">
-    <color rgba="0.0 0.8 0.0 1.0"/>
-  </material>
-  <material name="blue">
-    <color rgba="0.0 0.0 0.8 1.0"/>
-  </material>
-  <material name="black">
-    <color rgba="0 0 0 1"/>
-  </material>
-  <material name="white">
-    <color rgba="1 1 1 1"/>
-  </material>
-  <material name="orange">
-    <color rgba="1 0.3 0.1 1"/>
-  </material>
-  <material name="silver">
-    <color rgba="0.79 0.82 0.93 1"/>
-  </material>
-  <material name="dark_grey">
-    <color rgba="0.3 0.3 0.3 1"/>
-  </material>
-  <!-- Color adicional para ruedas -->
-  <material name="wheel_color">
-    <color rgba="0.6 0.6 0.6 1"/>
-  </material>
 </robot>

File: tp1_robot/urdf/motor.xacro (robot description, xacro)
@@ -1,72 +1,67 @@
 <?xml version="1.0"?>
-<robot xmlns:xacro="http://www.ros.org/wiki/xacro">
-  <!-- ======================= -->
-  <!-- === Macro de Motor === -->
-  <!-- ======================= -->
-  <!-- Este macro inserta un motor en el chasis del robot.
-       Se puede usar para ambos lados (izquierdo o derecho)
-       Parametrizado para posicionar correctamente el motor según el ancho del chasis.
-       Opcionalmente se puede reflejar para el lado derecho. -->
-  <!-- === Parámetros del macro === -->
-  <!-- prefix: prefijo para los nombres del link y joint (ej: left, right) -->
-  <!-- chassis_width: ancho total del chasis (usado para calcular posición Y del motor) -->
-  <!-- reflect: booleano que indica si el motor debe ser reflejado (para el lado derecho) -->
-  <xacro:macro name="motor" params="prefix chassis_width:=0 reflect:=false">
-    <!-- === Propiedades físicas del motor === -->
-    <!-- Masa del motor en kilogramos -->
-    <xacro:property name="motor_mass" value="0.1"/>
-    <!-- Dimensiones del motor en metros (x, y, z) -->
-    <xacro:property name="motor_x_size" value="0.07"/>
-    <xacro:property name="motor_y_size" value="0.0188"/>
-    <xacro:property name="motor_z_size" value="0.0225"/>
-    <!-- Desplazamiento del motor respecto al centro del chasis -->
-    <xacro:property name="motor_x_offset" value="0.0015"/>
-    <xacro:property name="motor_y_offset" value="0.0216"/>
-    <xacro:property name="motor_z_offset" value="-0.017"/>
-    <!-- Cálculo automático de posición Y del joint -->
-    <xacro:property name="pos_y_joint"
-      value="${(chassis_width / 2) - motor_y_offset + (motor_y_size / 2)}"/>
-    <!-- Posición fija del joint en X y Z -->
-    <xacro:property name="pos_x_joint" value="${motor_x_offset}"/>
-    <xacro:property name="pos_z_joint" value="${motor_z_offset}"/>
-    <!-- === Definición del link del motor === -->
-    <link name="${prefix}_motor">
-      <!-- === Visualización del motor === -->
+<robot xmlns:xacro="http://ros.org/wiki/xacro"
+       xmlns:gazebo="http://www.gazebosim.org/schema/gazebo_urdf">
+  <!-- Macro para insertar un motor con inercia -->
+  <xacro:macro name="motor" params="prefix chassis_width reflect">
+    <!-- Parámetros internos -->
+    <xacro:property name="motor_mass" value="0.1"/> <!-- Masa del motor (kg) -->
+    <xacro:property name="motor_length" value="0.07"/> <!-- Largo del motor (m) -->
+    <xacro:property name="motor_width" value="0.025"/> <!-- Ancho del motor (m) -->
+    <xacro:property name="motor_height" value="0.025"/> <!-- Altura del motor (m) -->
+    <xacro:property name="motor_radius" value="0.0125"/> <!-- Radio de los extremos (m) -->
+    <!-- Posición en X (ajustada según reflect) -->
+    <xacro:if value="${reflect}">
+      <xacro:property name="motor_x" value="${chassis_width/2 - 0.035}"/>
+    </xacro:if>
+    <xacro:unless value="${reflect}">
+      <xacro:property name="motor_x" value="${-chassis_width/2 + 0.035}"/>
+    </xacro:unless>
+    <!-- Link del motor -->
+    <link name="${prefix}_motor_link">
       <visual>
-        <origin xyz="0 0 0" rpy="0 0 0"/>
+        <origin xyz="${motor_x} -0.01 0" rpy="0 0 0"/>
         <geometry>
-          <!-- Si 'reflect' es true, escala negativo en Y para invertir orientación -->
-          <xacro:if value="${reflect}">
-            <mesh filename="file://$(find tp1_robot)/meshes/motor.stl" scale="1 -1 1"/>
-          </xacro:if>
-          <xacro:unless value="${reflect}">
-            <mesh filename="file://$(find tp1_robot)/meshes/motor.stl"/>
-          </xacro:unless>
+          <box size="${motor_length} ${motor_width} ${motor_height}"/>
         </geometry>
-        <material name="blue"/>
+        <material name="black"/>
       </visual>
-      <!-- === Colisión del motor (caja simple para simuladores) === -->
       <collision>
-        <origin xyz="0 0 0" rpy="0 0 0"/>
+        <origin xyz="${motor_x} -0.01 0" rpy="0 0 0"/>
         <geometry>
-          <box size="${motor_x_size} ${motor_y_size} ${motor_z_size}"/>
+          <box size="${motor_length} ${motor_width} ${motor_height}"/>
         </geometry>
       </collision>
-      <!-- === Inercia del motor (calculada automáticamente) === -->
-      <xacro:inertial_box mass="${motor_mass}" x="${motor_x_size}" y="${motor_y_size}" z="${motor_z_size}">
-        <origin xyz="0 0 0" rpy="0 0 0"/>
-      </xacro:inertial_box>
+      <!-- Usamos el macro box_inertia con el parámetro correcto 'm' -->
+      <xacro:box_inertia m="${motor_mass}" x="${motor_length}" y="${motor_width}" z="${motor_height}"/>
     </link>
-    <!-- === Joint fijo entre el chasis y el motor === -->
+    <!-- Joint del motor (fijo al chasis) -->
     <joint name="${prefix}_motor_joint" type="fixed">
       <parent link="base_link"/>
-      <child link="${prefix}_motor"/>
-      <!-- Posicionamiento dinámico del motor -->
-      <xacro:if value="${reflect}">
-        <origin xyz="${pos_x_joint} ${-1 * pos_y_joint} ${pos_z_joint}" rpy="0 0 0"/>
-      </xacro:if>
-      <xacro:unless value="${reflect}">
-        <origin xyz="${pos_x_joint} ${pos_y_joint} ${pos_z_joint}" rpy="0 0 0"/>
-      </xacro:unless>
+      <child link="${prefix}_motor_link"/>
+      <origin xyz="${motor_x} -0.01 0" rpy="0 0 0"/>
+    </joint>
+    <!-- Rotor del motor (simulado como cilindro) -->
+    <link name="${prefix}_motor_rotor_link">
+      <visual>
+        <origin xyz="0 0 0" rpy="0 1.5708 0"/>
+        <geometry>
+          <cylinder radius="${motor_radius}" length="${motor_width}"/>
+        </geometry>
+        <material name="gray"/>
+      </visual>
+      <collision>
+        <origin xyz="0 0 0" rpy="0 1.5708 0"/>
+        <geometry>
+          <cylinder radius="${motor_radius}" length="${motor_width}"/>
+        </geometry>
+      </collision>
+      <!-- Usamos el macro cylinder_inertia con el parámetro correcto 'm' -->
+      <xacro:cylinder_inertia m="${motor_mass/2}" r="${motor_radius}" h="${motor_width}"/>
+    </link>
+    <!-- Joint del rotor del motor (fijo al motor) -->
+    <joint name="${prefix}_motor_rotor_joint" type="fixed">
+      <parent link="${prefix}_motor_link"/>
+      <child link="${prefix}_motor_rotor_link"/>
+      <origin xyz="0 0 0" rpy="0 0 0"/>
     </joint>
   </xacro:macro>
