Commit message: tp1_robot_V0.15

File: tp1_robot/urdf/inertial_macros.xacro (robot description, xacro)
@@ -2,29 +2,50 @@
 <robot xmlns:xacro="http://ros.org/wiki/xacro"
        xmlns:gazebo="http://www.gazebosim.org/schema/gazebo_urdf">
-  <!-- Macro para inercia de un cilindro -->
-  <xacro:macro name="cylinder_inertia" params="m r h">
+    <!-- Macros de inercia -->
+    <xacro:macro name="inertial_sphere" params="mass radius origin">
+        <inertial>
+            <xacro:insert_block name="origin"/>
+            <mass value="${mass}"/>
+            <inertia ixx="${(2/5) * mass * (radius*radius)}" ixy="0.0" ixz="0.0"
+                     iyy="${(2/5) * mass * (radius*radius)}" iyz="0.0"
+                     izz="${(2/5) * mass * (radius*radius)}"/>
+        </inertial>
+    </xacro:macro>
+    <xacro:macro name="inertial_box" params="mass x y z">
     <inertial>
-      <mass value="${m}" />
-      <inertia
-        ixx="${m*(3*r*r + h*h)/12}"
-        ixy="0.0"
-        ixz="0.0"
-        iyy="${m*(3*r*r + h*h)/12}"
-        iyz="0.0"
-        izz="${m*r*r/2}" />
+        <origin xyz="0 0 0" rpy="0 0 0"/>
+        <mass value="${mass}"/>
+        <inertia ixx="${(1/12) * mass * (y*y + z*z)}" ixy="0.0" ixz="0.0"
+                iyy="${(1/12) * mass * (x*x + z*z)}" iyz="0.0"
+                izz="${(1/12) * mass * (x*x + y*y)}"/>
     </inertial>
-  </xacro:macro>
-  <!-- Macro para inercia de un cubo -->
-  <xacro:macro name="box_inertia" params="m x y z">
-    <inertial>
-      <mass value="${m}" />
-      <inertia
-        ixx="${m*(y*y + z*z)/6}"
-        ixy="0.0"
-        ixz="0.0"
-        iyy="${m*(x*x + z*z)/6}"
-        iyz="0.0"
-        izz="${m*(x*x + y*y)/6}" />
-    </inertial>
-  </xacro:macro>
+    </xacro:macro>
+    <xacro:macro name="inertial_cylinder" params="mass length radius origin">
+        <inertial>
+            <xacro:insert_block name="origin"/>
+            <mass value="${mass}"/>
+            <inertia ixx="${(1/12) * mass * (3*radius*radius + length*length)}" ixy="0.0" ixz="0.0"
+                     iyy="${(1/12) * mass * (3*radius*radius + length*length)}" iyz="0.0"
+                     izz="${(1/2) * mass * (radius*radius)}"/>
+        </inertial>
+    </xacro:macro>
+    <!-- Inercia dummy -->
+    <xacro:macro name="dummy_inertial">
+        <inertial>
+            <origin xyz="0 0 0" rpy="0 0 0"/>
+            <mass value="0.001"/>
+            <inertia ixx="0.00001" ixy="0" ixz="0"
+                     iyy="0.00001" iyz="0"
+                     izz="0.00001"/>
+        </inertial>
+    </xacro:macro>
+    <!-- Materiales -->
+    <material name="red"><color rgba="0.8 0.0 0.0 1.0"/></material>
+    <material name="green"><color rgba="0.0 0.8 0.0 1.0"/></material>
+    <material name="blue"><color rgba="0.0 0.0 0.8 1.0"/></material>
+    <material name="black"><color rgba="0 0 0 1"/></material>
+    <material name="white"><color rgba="1 1 1 1"/></material>
+    <material name="orange"><color rgba="1 0.3 0.1 1"/></material>
+    <material name="silver"><color rgba="0.79 0.82 0.93 1"/></material>
+    <material name="dark_grey"><color rgba="0.3 0.3 0.3 1"/></material>
 </robot>

File: tp1_robot/urdf/motor.xacro (robot description, xacro)
@@ -2,67 +2,54 @@
 <robot xmlns:xacro="http://ros.org/wiki/xacro"
        xmlns:gazebo="http://www.gazebosim.org/schema/gazebo_urdf">
-  <!-- Macro para insertar un motor con inercia -->
-  <xacro:macro name="motor" params="prefix chassis_width reflect">
-    <!-- Parámetros internos -->
-    <xacro:property name="motor_mass" value="0.1"/> <!-- Masa del motor (kg) -->
-    <xacro:property name="motor_length" value="0.07"/> <!-- Largo del motor (m) -->
-    <xacro:property name="motor_width" value="0.025"/> <!-- Ancho del motor (m) -->
-    <xacro:property name="motor_height" value="0.025"/> <!-- Altura del motor (m) -->
-    <xacro:property name="motor_radius" value="0.0125"/> <!-- Radio de los extremos (m) -->
-    <!-- Posición en X (ajustada según reflect) -->
-    <xacro:if value="${reflect}">
-      <xacro:property name="motor_x" value="${chassis_width/2 - 0.035}"/>
-    </xacro:if>
-    <xacro:unless value="${reflect}">
-      <xacro:property name="motor_x" value="${-chassis_width/2 + 0.035}"/>
-    </xacro:unless>
-    <!-- Link del motor -->
-    <link name="${prefix}_motor_link">
-      <visual>
-        <origin xyz="${motor_x} -0.01 0" rpy="0 0 0"/>
-        <geometry>
-          <box size="${motor_length} ${motor_width} ${motor_height}"/>
-        </geometry>
-        <material name="black"/>
-      </visual>
-      <collision>
-        <origin xyz="${motor_x} -0.01 0" rpy="0 0 0"/>
-        <geometry>
-          <box size="${motor_length} ${motor_width} ${motor_height}"/>
-        </geometry>
-      </collision>
-      <!-- Usamos el macro box_inertia con el parámetro correcto 'm' -->
-      <xacro:box_inertia m="${motor_mass}" x="${motor_length}" y="${motor_width}" z="${motor_height}"/>
-    </link>
-    <!-- Joint del motor (fijo al chasis) -->
-    <joint name="${prefix}_motor_joint" type="fixed">
-      <parent link="base_link"/>
-      <child link="${prefix}_motor_link"/>
-      <origin xyz="${motor_x} -0.01 0" rpy="0 0 0"/>
-    </joint>
-    <!-- Rotor del motor (simulado como cilindro) -->
-    <link name="${prefix}_motor_rotor_link">
-      <visual>
-        <origin xyz="0 0 0" rpy="0 1.5708 0"/>
-        <geometry>
-          <cylinder radius="${motor_radius}" length="${motor_width}"/>
-        </geometry>
-        <material name="gray"/>
-      </visual>
-      <collision>
-        <origin xyz="0 0 0" rpy="0 1.5708 0"/>
-        <geometry>
-          <cylinder radius="${motor_radius}" length="${motor_width}"/>
-        </geometry>
-      </collision>
-      <!-- Usamos el macro cylinder_inertia con el parámetro correcto 'm' -->
-      <xacro:cylinder_inertia m="${motor_mass/2}" r="${motor_radius}" h="${motor_width}"/>
-    </link>
-    <!-- Joint del rotor del motor (fijo al motor) -->
-    <joint name="${prefix}_motor_rotor_joint" type="fixed">
-      <parent link="${prefix}_motor_link"/>
-      <child link="${prefix}_motor_rotor_link"/>
-      <origin xyz="0 0 0" rpy="0 0 0"/>
-    </joint>
-  </xacro:macro>
+    <xacro:macro name="motor" params="prefix chassis_width:=0 reflect:=false">
+        <!-- Parámetros -->
+        <xacro:property name="motor_mass" value="0.1"/>
+        <xacro:property name="motor_x_size" value="0.07"/>
+        <xacro:property name="motor_y_size" value="0.0188"/>
+        <xacro:property name="motor_z_size" value="0.0225"/>
+        <xacro:property name="motor_x_offset" value="0.0015"/>
+        <xacro:property name="motor_y_offset" value="0.0216"/>
+        <xacro:property name="motor_z_offset" value="-0.017"/>
+        <xacro:property name="pos_x_joint" value="${motor_x_offset}"/>
+        <xacro:property name="pos_y_joint" value="${(chassis_width/2) - motor_y_offset + (motor_y_size/2)}"/>
+        <xacro:property name="pos_z_joint" value="${motor_z_offset}"/>
+        <!-- Link del motor -->
+        <link name="${prefix}_motor">
+            <!-- Visual -->
+            <visual>
+                <origin xyz="0 0 0" rpy="0 0 0"/>
+                <geometry>
+                    <xacro:if value="${reflect}">
+                        <mesh filename="file://$(find tp1_robot)/meshes/motor.stl" scale="1 -1 1"/>
+                    </xacro:if>
+                    <xacro:unless value="${reflect}">
+                        <mesh filename="file://$(find tp1_robot)/meshes/motor.stl"/>
+                    </xacro:unless>
+                </geometry>
+                <material name="blue"/>
+            </visual>
+            <!-- Colisión -->
+            <collision>
+                <origin xyz="0 0 0" rpy="0 0 0"/>
+                <geometry>
+                    <box size="${motor_x_size} ${motor_y_size} ${motor_z_size}"/>
+                </geometry>
+            </collision>
+            <!-- Inercia -->
+            <xacro:inertial_box mass="${motor_mass}" x="${motor_x_size}" y="${motor_y_size}" z="${motor_z_size}">
+                <!-- <origin xyz="0 0 0" rpy="0 0 0"/>-->
+            </xacro:inertial_box>
+        </link>
+        <!-- Joint del motor -->
+        <joint name="${prefix}_motor_joint" type="fixed">
+            <parent link="base_link"/>
+            <child link="${prefix}_motor"/>
+            <xacro:if value="${reflect}">
+                <origin xyz="${pos_x_joint} ${-1 * pos_y_joint} ${pos_z_joint}" rpy="0 0 0"/>
+            </xacro:if>
+            <xacro:unless value="${reflect}">
+                <origin xyz="${pos_x_joint} ${pos_y_joint} ${pos_z_joint}" rpy="0 0 0"/>
+            </xacro:unless>
+        </joint>
+    </xacro:macro>
 </robot>
