Commit message: tp1_robot_V0.4

File: tp1_robot/urdf/diffbot.urdf.xacro (robot description, xacro)
@@ -22,20 +22,23 @@
     </link>
     <!-- Macro de ruedas -->
-    <xacro:macro name="wheel" params="prefix side">
-        <link name="${prefix}_wheel">
-            <visual>
-                <geometry><cylinder radius="0.035" length="0.025"/></geometry>
-            </visual>
-        </link>
-        <joint name="${prefix}_wheel_joint" type="continuous">
-            <parent link="base_link"/>
-            <child link="${prefix}_wheel"/>
-            <axis xyz="0 1 0"/>
-            <origin xyz="0.0625 ${side*0.08} -0.025"/>
-        </joint>
+    <xacro:macro name="wheel" params="prefix side xyz rpy">
+    <link name="${prefix}_wheel">
+        <visual>
+        <geometry><cylinder radius="0.035" length="0.025"/></geometry>
+        </visual>
+    </link>
+    <joint name="${prefix}_wheel_joint" type="continuous">
+        <parent link="base_link"/>
+        <child link="${prefix}_wheel"/>
+        <axis xyz="0 1 0"/>
+        <origin xyz="${xyz}" rpy="${rpy}"/>
+    </joint>
     </xacro:macro>
     <!-- Instanciar ruedas y motores -->
-    <xacro:wheel prefix="left" side="1"/>
-    <xacro:wheel prefix="right" side="-1"/>
+    <!-- <xacro:wheel prefix="left" side="1"/>
+        <xacro:wheel prefix="right" side="-1"/> -->
+    <!-- Ejemplo con nueva posición y rotación xyz="0.0625 0.08 -0.025" -->
+    <xacro:wheel prefix="left"  side="1"  xyz="0 0.08 -0.025"  rpy="0 0 1.5708"/>
+    <xacro:wheel prefix="right" side="-1" xyz="0 -0.08 -0.025" rpy="0 0 1.5708"/>
     <xacro:motor prefix="left" chassis_width="0.1" reflect="false"/>
     <xacro:motor prefix="right" chassis_width="0.1" reflect="true"/>

Commit message: tp1_robot_V0.5

File: tp1_robot/urdf/diffbot.urdf.xacro (robot description, xacro)
@@ -22,14 +22,23 @@
     </link>
     <!-- Macro de ruedas -->
-    <xacro:macro name="wheel" params="prefix side xyz rpy">
+    <xacro:macro name="wheel" params="prefix side xyz rpy axis">
     <link name="${prefix}_wheel">
         <visual>
-        <geometry><cylinder radius="0.035" length="0.025"/></geometry>
+        <origin rpy="1.5708 0 0"/> <!-- Rotación de 90° en X -->
+        <geometry>
+            <cylinder radius="0.035" length="0.025"/>
+        </geometry>
         </visual>
+        <collision>
+        <origin rpy="1.5708 0 0"/> <!-- También rotamos para colisiones -->
+        <geometry>
+            <cylinder radius="0.035" length="0.025"/>
+        </geometry>
+        </collision>
     </link>
     <joint name="${prefix}_wheel_joint" type="continuous">
         <parent link="base_link"/>
         <child link="${prefix}_wheel"/>
-        <axis xyz="0 1 0"/>
+        <axis xyz="${axis}"/>
         <origin xyz="${xyz}" rpy="${rpy}"/>
     </joint>
@@ -39,6 +48,6 @@
         <xacro:wheel prefix="right" side="-1"/> -->
     <!-- Ejemplo con nueva posición y rotación xyz="0.0625 0.08 -0.025" -->
-    <xacro:wheel prefix="left"  side="1"  xyz="0 0.08 -0.025"  rpy="0 0 1.5708"/>
-    <xacro:wheel prefix="right" side="-1" xyz="0 -0.08 -0.025" rpy="0 0 1.5708"/>
+    <xacro:wheel prefix="left"  side="1"  xyz="-0.0625 0.08 -0.025"  rpy="0 0 0" axis="0 1 0"/>
+    <xacro:wheel prefix="right" side="-1" xyz="-0.0625 -0.08 -0.025" rpy="0 0 0" axis="0 1 0"/>
     <xacro:motor prefix="left" chassis_width="0.1" reflect="false"/>
     <xacro:motor prefix="right" chassis_width="0.1" reflect="true"/>

Commit message: 13062025V1

File: tp1_robot/urdf/diffbot.urdf.xacro (robot description, xacro)
@@ -95,4 +95,14 @@
       <material name="${caster_color}"/>
     </visual>
+    <collision>
+      <origin xyz="0 0 0.0045" rpy="0 0 0"/>
+      <geometry>
+        <box size="0.05 0.05 0.01"/>
+      </geometry>
+    </collision>
+    <inertial>
+      <mass value="0.1"/>
+      <inertia ixx="0.001" ixy="0" ixz="0" iyy="0.001" iyz="0" izz="0.001"/>
+    </inertial>
   </link>
   <joint name="caster_joint" type="fixed">
@@ -109,4 +119,14 @@
       <material name="${caster_color}"/>
     </visual>
+    <collision>
+      <origin xyz="-0.015 0 -0.020" rpy="0 0 0"/>
+      <geometry>
+        <cylinder radius="0.02" length="0.01"/>
+      </geometry>
+    </collision>
+    <inertial>
+      <mass value="0.1"/>
+      <inertia ixx="0.001" ixy="0" ixz="0" iyy="0.001" iyz="0" izz="0.001"/>
+    </inertial>
   </link>
   <joint name="caster_wheel_joint" type="continuous">
@@ -124,4 +144,14 @@
       <material name="${caster_color}"/>
     </visual>
+    <collision>
+      <origin xyz="0 0 0" rpy="0 0 0"/>
+      <geometry>
+        <box size="0.02 0.02 0.02"/>
+      </geometry>
+    </collision>
+    <inertial>
+      <mass value="0.1"/>
+      <inertia ixx="0.001" ixy="0" ixz="0" iyy="0.001" iyz="0" izz="0.001"/>
+    </inertial>
   </link>
   <joint name="caster_support_joint" type="fixed">
@@ -130,4 +160,16 @@
     <origin xyz="0 0 0" rpy="0 0 0"/>
   </joint>
+  <!-- Gazebo properties for caster components -->
+  <gazebo reference="caster">
+    <material>Gazebo/Orange</material>
+  </gazebo>
+  <gazebo reference="caster_wheel">
+    <material>Gazebo/Orange</material>
+    <mu1>1.0</mu1>
+    <mu2>1.0</mu2>
+  </gazebo>
+  <gazebo reference="caster_wheel_support">
+    <material>Gazebo/Orange</material>
+  </gazebo>
   <!-- ======================= -->
   <!-- === Frame odométrico === -->
@@ -144,5 +186,5 @@
   <ros2_control name="DiffbotSystemHardware" type="system">
     <hardware>
-      <plugin>gz_ros2_control/DefaultSystem</plugin>
+      <plugin>mock_components/GenericSystem</plugin>
     </hardware>
     <joint name="left_wheel_joint">
@@ -165,5 +207,5 @@
   <!-- ============================ -->
   <gazebo>
-    <plugin name="gz_ros2_control" filename="libgz_ros2_control.so">
+    <plugin name="gz_ros2_control" filename="libgz_ros2_control_system.so">
       <ros2_control_parameters>$(find tp1_robot)/config/diffbot_controllers.yaml</ros2_control_parameters>
     </plugin>

Commit message: 13062025V2
Correxion xacro ruedas laterales y medidas generales. Ya se ve en gazebo

File: tp1_robot/urdf/diffbot.urdf.xacro (robot description, xacro)
@@ -7,9 +7,9 @@
   <!-- ======================= -->
   <xacro:property name="chassis_mass" value="0.8"/>
-  <xacro:property name="wheel_radius" value="0.035"/>
-  <xacro:property name="wheel_width" value="0.025"/>
-  <xacro:property name="wheel_separation" value="0.16"/>
+  <xacro:property name="wheel_radius" value="0.035"/> <!-- Radio de la rueda en metros -->
+  <xacro:property name="wheel_width" value="0.025"/> <!-- Ancho de la rueda en metros -->
+  <xacro:property name="wheel_separation" value="0.16"/> <!-- Separación entre ruedas en metros -->
   <xacro:property name="wheel_color" value="silver"/>
-  <xacro:property name="caster_origin_xyz" value="-0.075 0 0.002"/>
+  <xacro:property name="caster_origin_xyz" value="-0.075 0 -0.0015"/> <!-- Posición del caster respecto al chasis (x: atrás, y: centro, z: altura) -->
   <xacro:property name="caster_color" value="orange"/>
   <!-- ======================= -->
@@ -23,5 +23,4 @@
   <link name="base_link">
     <visual>
-      <!-- <origin xyz="0 0 0" rpy="0 0 0"/>-->
       <geometry>
         <mesh filename="file://$(find tp1_robot)/meshes/chassis.stl"/>
@@ -29,7 +28,6 @@
     </visual>
     <collision>
-      <!-- <origin xyz="0 0 0" rpy="0 0 0"/>-->
-      <geometry>
-        <box size="0.195 0.1 0.05"/>
+      <geometry>
+        <box size="0.195 0.1 0.05"/> <!-- Tamaño del chasis (x: largo, y: ancho, z: alto) -->
       </geometry>
     </collision>
@@ -39,15 +37,15 @@
   <!-- === Macro para ruedas === -->
   <!-- ======================= -->
-  <xacro:macro name="wheel" params="prefix xyz axis">
+  <xacro:macro name="wheel" params="prefix xyz axis rpy">
     <link name="${prefix}_wheel">
       <visual>
-        <origin xyz="0 0 0" rpy="1.5708 0 0"/>
+        <origin xyz="0 0 0" rpy="1.5708 0 0"/> <!-- Origen de la visualización de la rueda -->
         <geometry>
-          <cylinder radius="${wheel_radius}" length="${wheel_width}"/>
+          <mesh filename="file://$(find tp1_robot)/meshes/wheel.stl"/>
         </geometry>
         <material name="${wheel_color}"/>
       </visual>
       <collision>
-        <origin xyz="0 0 0" rpy="1.5708 0 0"/>
+        <origin xyz="0 0 0" rpy="1.5708 0 0"/> <!-- Origen de la colisión de la rueda -->
         <geometry>
           <cylinder radius="${wheel_radius}" length="${wheel_width}"/>
@@ -56,5 +54,5 @@
       <inertial>
         <mass value="0.2"/>
-        <origin xyz="0 0 0" rpy="0 0 0"/>
+        <origin xyz="0 0 0" rpy="0 0 0"/> <!-- Centro de masa de la rueda -->
         <inertia ixx="0.001" ixy="0.0" ixz="0.0"
                  iyy="0.001" iyz="0.0"
@@ -63,5 +61,5 @@
     </link>
     <joint name="${prefix}_wheel_joint" type="continuous">
-      <origin xyz="${xyz}" rpy="0 0 0"/>
+      <origin xyz="${xyz}" rpy="${rpy}"/> <!-- Posición de la rueda respecto al chasis (x: adelante/atrás, y: izquierda/derecha, z: arriba/abajo) -->
       <parent link="base_link"/>
       <child link="${prefix}_wheel"/>
@@ -80,6 +78,6 @@
   <!-- === Ruedas y motores === -->
   <!-- ======================= -->
-  <xacro:wheel prefix="left"  xyz="0.0175  0.065 -0.0175" axis="0 1 0"/>
-  <xacro:wheel prefix="right" xyz="0.0175 -0.065 -0.0175" axis="0 1 0"/>
+  <xacro:wheel prefix="left"  xyz="0.0185  0.05 -0.0175" axis="0 1 0" rpy="0 1.5708 0"/> <!-- Rueda izquierda (x: adelante, y: izquierda, z: abajo) -->
+  <xacro:wheel prefix="right" xyz="0.0185 -0.05 -0.0175" axis="0 1 0" rpy="0 1.5708 3.14159"/> <!-- Rueda derecha (x: adelante, y: derecha, z: abajo) -->
   <xacro:motor prefix="left" chassis_width="0.1" reflect="false"/>
   <xacro:motor prefix="right" chassis_width="0.1" reflect="true"/>
@@ -89,5 +87,5 @@
   <link name="caster">
     <visual>
-      <origin xyz="0 0 0.0045" rpy="0 0 0"/>
+      <origin xyz="0 0 0.0045" rpy="0 0 0"/> <!-- Origen de la visualización del caster -->
       <geometry>
         <mesh filename="file://$(find tp1_robot)/meshes/caster_base.stl"/>
@@ -96,7 +94,7 @@
     </visual>
     <collision>
-      <origin xyz="0 0 0.0045" rpy="0 0 0"/>
-      <geometry>
-        <box size="0.05 0.05 0.01"/>
+      <origin xyz="0 0 0.0045" rpy="0 0 0"/> <!-- Origen de la colisión del caster -->
+      <geometry>
+        <box size="0.05 0.05 0.01"/> <!-- Tamaño del caster (x: largo, y: ancho, z: alto) -->
       </geometry>
     </collision>
@@ -109,9 +107,9 @@
     <parent link="base_link"/>
     <child link="caster"/>
-    <origin xyz="${caster_origin_xyz}" rpy="0 0 0"/>
+    <origin xyz="${caster_origin_xyz}" rpy="0 0 0"/> <!-- Posición del caster respecto al chasis -->
   </joint>
   <link name="caster_wheel">
     <visual>
-      <origin xyz="-0.015 0 -0.020" rpy="0 0 0"/>
+      <origin xyz="-0.015 0 -0.020" rpy="0 0 0"/> <!-- Origen de la visualización de la rueda del caster -->
       <geometry>
         <mesh filename="file://$(find tp1_robot)/meshes/caster_wheel.stl"/>
@@ -120,7 +118,7 @@
     </visual>
     <collision>
-      <origin xyz="-0.015 0 -0.020" rpy="0 0 0"/>
-      <geometry>
-        <cylinder radius="0.02" length="0.01"/>
+      <origin xyz="-0.015 0 -0.020" rpy="0 0 0"/> <!-- Origen de la colisión de la rueda del caster -->
+      <geometry>
+        <cylinder radius="0.02" length="0.01"/> <!-- Radio y longitud de la rueda del caster -->
       </geometry>
     </collision>
@@ -133,10 +131,10 @@
     <parent link="caster"/>
     <child link="caster_wheel"/>
-    <origin xyz="0 0 -0.01" rpy="0 0 0"/>
+    <origin xyz="0 0 -0.01" rpy="0 0 0"/> <!-- Posición de la rueda del caster respecto al caster -->
     <axis xyz="0 0 1"/>
   </joint>
   <link name="caster_wheel_support">
     <visual>
-      <origin xyz="0 0 0" rpy="0 0 0"/>
+      <origin xyz="0 0 0" rpy="0 0 0"/> <!-- Origen de la visualización del soporte del caster -->
       <geometry>
         <mesh filename="file://$(find tp1_robot)/meshes/caster_wheel_support.stl"/>
@@ -145,7 +143,7 @@
     </visual>
     <collision>
-      <origin xyz="0 0 0" rpy="0 0 0"/>
-      <geometry>
-        <box size="0.02 0.02 0.02"/>
+      <origin xyz="0 0 0" rpy="0 0 0"/> <!-- Origen de la colisión del soporte del caster -->
+      <geometry>
+        <box size="0.02 0.02 0.02"/> <!-- Tamaño del soporte del caster (x: largo, y: ancho, z: alto) -->
       </geometry>
     </collision>

Commit message: 13062025V3
Correcion rueda trasera

File: tp1_robot/urdf/diffbot.urdf.xacro (robot description, xacro)
@@ -118,5 +118,5 @@
     </visual>
     <collision>
-      <origin xyz="-0.015 0 -0.020" rpy="0 0 0"/> <!-- Origen de la colisión de la rueda del caster -->
+      <origin xyz="-0.015 0 -0.030" rpy="0 0 0"/> <!-- Origen de la colisión de la rueda del caster (Modificar colicion rueda giro)-->
       <geometry>
         <cylinder radius="0.02" length="0.01"/> <!-- Radio y longitud de la rueda del caster -->
