Commit message: 20062025

File: tp1_robot/urdf/diffbot.urdf.xacro (robot description, xacro)
@@ -6,10 +6,11 @@
   <!-- === Propiedades === -->
   <!-- ======================= -->
-  <xacro:property name="chassis_mass" value="0.8"/>
+  <xacro:property name="chassis_mass" value="0.800"/>
+  <xacro:property name="base_color" value="green"/>
   <xacro:property name="wheel_radius" value="0.035"/> <!-- Radio de la rueda en metros -->
   <xacro:property name="wheel_width" value="0.025"/> <!-- Ancho de la rueda en metros -->
   <xacro:property name="wheel_separation" value="0.16"/> <!-- Separación entre ruedas en metros -->
   <xacro:property name="wheel_color" value="silver"/>
-  <xacro:property name="caster_origin_xyz" value="-0.075 0 -0.0015"/> <!-- Posición del caster respecto al chasis (x: atrás, y: centro, z: altura) -->
+  <xacro:property name="caster_origin_xyz" value="-0.075 0 -0.0075"/> <!-- Posición del caster respecto al chasis -->
   <xacro:property name="caster_color" value="orange"/>
   <!-- ======================= -->
@@ -26,4 +27,5 @@
         <mesh filename="file://$(find tp1_robot)/meshes/chassis.stl"/>
       </geometry>
+      <material name="${base_color}"/>
     </visual>
     <collision>
@@ -40,5 +42,5 @@
     <link name="${prefix}_wheel">
       <visual>
-        <origin xyz="0 0 0" rpy="1.5708 0 0"/> <!-- Origen de la visualización de la rueda -->
+        <origin xyz="0 0 0" rpy="1.5708 0 0"/>
         <geometry>
           <mesh filename="file://$(find tp1_robot)/meshes/wheel.stl"/>
@@ -47,19 +49,15 @@
       </visual>
       <collision>
-        <origin xyz="0 0 0" rpy="1.5708 0 0"/> <!-- Origen de la colisión de la rueda -->
+        <origin xyz="0 0 0" rpy="1.5708 0 0"/>
         <geometry>
           <cylinder radius="${wheel_radius}" length="${wheel_width}"/>
         </geometry>
       </collision>
-      <inertial>
-        <mass value="0.2"/>
-        <origin xyz="0 0 0" rpy="0 0 0"/> <!-- Centro de masa de la rueda -->
-        <inertia ixx="0.001" ixy="0.0" ixz="0.0"
-                 iyy="0.001" iyz="0.0"
-                 izz="0.001"/>
-      </inertial>
+      <xacro:inertial_cylinder mass="0.150" radius="${wheel_radius}" length="${wheel_width}">
+        <origin xyz="0 0 0" rpy="0 0 0"/>
+      </xacro:inertial_cylinder>
     </link>
     <joint name="${prefix}_wheel_joint" type="continuous">
-      <origin xyz="${xyz}" rpy="${rpy}"/> <!-- Posición de la rueda respecto al chasis (x: adelante/atrás, y: izquierda/derecha, z: arriba/abajo) -->
+      <origin xyz="${xyz}" rpy="${rpy}"/>
       <parent link="base_link"/>
       <child link="${prefix}_wheel"/>
@@ -78,6 +76,6 @@
   <!-- === Ruedas y motores === -->
   <!-- ======================= -->
-  <xacro:wheel prefix="left"  xyz="0.0185  0.05 -0.0175" axis="0 1 0" rpy="0 1.5708 0"/> <!-- Rueda izquierda (x: adelante, y: izquierda, z: abajo) -->
-  <xacro:wheel prefix="right" xyz="0.0185 -0.05 -0.0175" axis="0 1 0" rpy="0 1.5708 3.14159"/> <!-- Rueda derecha (x: adelante, y: derecha, z: abajo) -->
+  <xacro:wheel prefix="left" xyz="0.0185  0.05 -0.0175" axis="0 1 0" rpy="0 1.5708 0"/>
+  <xacro:wheel prefix="right" xyz="0.0185 -0.05 -0.0175" axis="0 1 0" rpy="0 1.5708 3.14159"/>
   <xacro:motor prefix="left" chassis_width="0.1" reflect="false"/>
   <xacro:motor prefix="right" chassis_width="0.1" reflect="true"/>
@@ -100,5 +98,5 @@
     </collision>
     <inertial>
-      <mass value="0.1"/>
+      <mass value="0.020"/>
       <inertia ixx="0.001" ixy="0" ixz="0" iyy="0.001" iyz="0" izz="0.001"/>
     </inertial>
@@ -107,9 +105,9 @@
     <parent link="base_link"/>
     <child link="caster"/>
-    <origin xyz="${caster_origin_xyz}" rpy="0 0 0"/> <!-- Posición del caster respecto al chasis -->
+    <origin xyz="${caster_origin_xyz}" rpy="0 0 0"/>
   </joint>
   <link name="caster_wheel">
     <visual>
-      <origin xyz="-0.015 0 -0.020" rpy="0 0 0"/> <!-- Origen de la visualización de la rueda del caster -->
+      <origin xyz="-0.015 0 -0.020" rpy="0 0 0"/>
       <geometry>
         <mesh filename="file://$(find tp1_robot)/meshes/caster_wheel.stl"/>
@@ -118,18 +116,17 @@
     </visual>
     <collision>
-      <origin xyz="-0.015 0 -0.030" rpy="0 0 0"/> <!-- Origen de la colisión de la rueda del caster (Modificar colicion rueda giro)-->
-      <geometry>
-        <cylinder radius="0.02" length="0.01"/> <!-- Radio y longitud de la rueda del caster -->
-      </geometry>
-    </collision>
-    <inertial>
-      <mass value="0.1"/>
-      <inertia ixx="0.001" ixy="0" ixz="0" iyy="0.001" iyz="0" izz="0.001"/>
-    </inertial>
+      <origin xyz="-0.015 0 -0.030" rpy="0 0 0"/>
+      <geometry>
+        <cylinder radius="0.02" length="0.01"/>
+      </geometry>
+    </collision>
+    <xacro:inertial_cylinder mass="0.150" radius="0.015" length="0.015">
+      <origin xyz="-0.015 0 -0.030" rpy="0 0 0"/>
+    </xacro:inertial_cylinder>
   </link>
   <joint name="caster_wheel_joint" type="continuous">
     <parent link="caster"/>
     <child link="caster_wheel"/>
-    <origin xyz="0 0 -0.01" rpy="0 0 0"/> <!-- Posición de la rueda del caster respecto al caster -->
+    <origin xyz="0 0 -0.01" rpy="0 0 0"/>
     <axis xyz="0 0 1"/>
   </joint>
@@ -149,5 +146,5 @@
     </collision>
     <inertial>
-      <mass value="0.1"/>
+      <mass value="0.020"/>
       <inertia ixx="0.001" ixy="0" ixz="0" iyy="0.001" iyz="0" izz="0.001"/>
     </inertial>
@@ -158,16 +155,4 @@
     <origin xyz="0 0 0" rpy="0 0 0"/>
   </joint>
-  <!-- Gazebo properties for caster components -->
-  <gazebo reference="caster">
-    <material>Gazebo/Orange</material>
-  </gazebo>
-  <gazebo reference="caster_wheel">
-    <material>Gazebo/Orange</material>
-    <mu1>1.0</mu1>
-    <mu2>1.0</mu2>
-  </gazebo>
-  <gazebo reference="caster_wheel_support">
-    <material>Gazebo/Orange</material>
-  </gazebo>
   <!-- ======================= -->
   <!-- === Frame odométrico === -->
@@ -205,5 +190,5 @@
   <!-- ============================ -->
   <gazebo>
-    <plugin name="gz_ros2_control" filename="libgz_ros2_control_system.so">
+    <plugin name="gz_ros2_control" filename="libgz_ros2_control.so">
       <ros2_control_parameters>$(find tp1_robot)/config/diffbot_controllers.yaml</ros2_control_parameters>
     </plugin>

File: tp1_robot/urdf/inertial_macros.xacro (robot description, xacro)
@@ -1,34 +1,33 @@
 <?xml version="1.0"?>
-<robot xmlns:xacro="http://ros.org/wiki/xacro"
-       xmlns:gazebo="http://www.gazebosim.org/schema/gazebo_urdf">
-    <!-- Macros de inercia -->
-    <xacro:macro name="inertial_sphere" params="mass radius origin">
+<robot xmlns:xacro="http://www.ros.org/wiki/xacro" >
+    <!-- Specify some standard inertial calculations https://en.wikipedia.org/wiki/List_of_moments_of_inertia -->
+    <!-- These make use of xacro's mathematical functionality -->
+    <xacro:macro name="inertial_sphere" params="mass radius *origin">
         <inertial>
             <xacro:insert_block name="origin"/>
-            <mass value="${mass}"/>
+            <mass value="${mass}" />
             <inertia ixx="${(2/5) * mass * (radius*radius)}" ixy="0.0" ixz="0.0"
-                     iyy="${(2/5) * mass * (radius*radius)}" iyz="0.0"
-                     izz="${(2/5) * mass * (radius*radius)}"/>
+                    iyy="${(2/5) * mass * (radius*radius)}" iyz="0.0"
+                    izz="${(2/5) * mass * (radius*radius)}" />
         </inertial>
     </xacro:macro>
     <xacro:macro name="inertial_box" params="mass x y z">
-    <inertial>
-        <origin xyz="0 0 0" rpy="0 0 0"/>
-        <mass value="${mass}"/>
-        <inertia ixx="${(1/12) * mass * (y*y + z*z)}" ixy="0.0" ixz="0.0"
-                iyy="${(1/12) * mass * (x*x + z*z)}" iyz="0.0"
-                izz="${(1/12) * mass * (x*x + y*y)}"/>
-    </inertial>
+        <inertial>
+            <origin xyz="0 0 0" rpy="0 0 0"/>
+            <mass value="${mass}"/>
+            <inertia ixx="${(1/12) * mass * (y*y + z*z)}" ixy="0.0" ixz="0.0"
+                    iyy="${(1/12) * mass * (x*x + z*z)}" iyz="0.0"
+                    izz="${(1/12) * mass * (x*x + y*y)}"/>
+        </inertial>
     </xacro:macro>
-    <xacro:macro name="inertial_cylinder" params="mass length radius origin">
+    <xacro:macro name="inertial_cylinder" params="mass length radius *origin">
         <inertial>
             <xacro:insert_block name="origin"/>
-            <mass value="${mass}"/>
+            <mass value="${mass}" />
             <inertia ixx="${(1/12) * mass * (3*radius*radius + length*length)}" ixy="0.0" ixz="0.0"
-                     iyy="${(1/12) * mass * (3*radius*radius + length*length)}" iyz="0.0"
-                     izz="${(1/2) * mass * (radius*radius)}"/>
+                    iyy="${(1/12) * mass * (3*radius*radius + length*length)}" iyz="0.0"
+                    izz="${(1/2) * mass * (radius*radius)}" />
         </inertial>
     </xacro:macro>
-    <!-- Inercia dummy -->
     <xacro:macro name="dummy_inertial">
         <inertial>
@@ -40,12 +39,28 @@
         </inertial>
     </xacro:macro>
-    <!-- Materiales -->
-    <material name="red"><color rgba="0.8 0.0 0.0 1.0"/></material>
-    <material name="green"><color rgba="0.0 0.8 0.0 1.0"/></material>
-    <material name="blue"><color rgba="0.0 0.0 0.8 1.0"/></material>
-    <material name="black"><color rgba="0 0 0 1"/></material>
-    <material name="white"><color rgba="1 1 1 1"/></material>
-    <material name="orange"><color rgba="1 0.3 0.1 1"/></material>
-    <material name="silver"><color rgba="0.79 0.82 0.93 1"/></material>
-    <material name="dark_grey"><color rgba="0.3 0.3 0.3 1"/></material>
+    <!-- RVIZ material RGBA definition -->
+    <material name="red">
+        <color rgba="0.8 0.0 0.0 1.0"/>
+    </material>
+    <material name="green">
+        <color rgba="0.0 0.8 0.0 1.0"/>
+    </material>
+    <material name="blue">
+        <color rgba="0.0 0.0 0.8 1.0"/>
+    </material>
+    <material name="black">
+        <color rgba="0 0 0 1"/>
+    </material>
+    <material name="white">
+        <color rgba="1 1 1 1"/>
+    </material>
+    <material name="orange">
+        <color rgba="1 0.3 0.1 1"/>
+    </material>
+    <material name="silver">
+        <color rgba="0.79 0.82 0.93 1"/>
+    </material>
+    <material name="dark_grey">
+        <color rgba="0.3 0.3 0.3 1"/>
+    </material>
 </robot>

Commit message: 22062025V2

File: tp1_robot/urdf/diffbot.urdf.xacro (robot description, xacro)
@@ -70,5 +70,5 @@
       <mu1>1.0</mu1>
       <mu2>1.0</mu2>
-      <material>Gazebo/Grey</material>
+      <!--<material>Gazebo/Grey</material>-->
     </gazebo>
   </xacro:macro>

Commit message: 22062025V3

File: tp1_robot/urdf/diffbot.urdf.xacro (robot description, xacro)
@@ -53,4 +53,12 @@
           <cylinder radius="${wheel_radius}" length="${wheel_width}"/>
         </geometry>
+        <!-- Movimos el contacto aquí -->
+        <contact>
+          <ode>
+            <min_depth>0.001</min_depth>
+            <kp>1e3</kp>
+            <kd>1e1</kd>
+          </ode>
+        </contact>
       </collision>
       <xacro:inertial_cylinder mass="0.150" radius="${wheel_radius}" length="${wheel_width}">
@@ -70,5 +78,5 @@
       <mu1>1.0</mu1>
       <mu2>1.0</mu2>
-      <!--<material>Gazebo/Grey</material>-->
+      <material>Gazebo/Grey</material>
     </gazebo>
   </xacro:macro>
@@ -85,5 +93,5 @@
   <link name="caster">
     <visual>
-      <origin xyz="0 0 0.0045" rpy="0 0 0"/> <!-- Origen de la visualización del caster -->
+      <origin xyz="0 0 0.0045" rpy="0 0 0"/>
       <geometry>
         <mesh filename="file://$(find tp1_robot)/meshes/caster_base.stl"/>
@@ -92,7 +100,7 @@
     </visual>
     <collision>
-      <origin xyz="0 0 0.0045" rpy="0 0 0"/> <!-- Origen de la colisión del caster -->
-      <geometry>
-        <box size="0.05 0.05 0.01"/> <!-- Tamaño del caster (x: largo, y: ancho, z: alto) -->
+      <origin xyz="0 0 0.0045" rpy="0 0 0"/>
+      <geometry>
+        <box size="0.05 0.05 0.01"/>
       </geometry>
     </collision>
@@ -120,4 +128,12 @@
         <cylinder radius="0.02" length="0.01"/>
       </geometry>
+      <!-- Contacto también aquí si lo necesitas -->
+      <contact>
+        <ode>
+          <min_depth>0.001</min_depth>
+          <kp>1e3</kp>
+          <kd>1e1</kd>
+        </ode>
+      </contact>
     </collision>
     <xacro:inertial_cylinder mass="0.150" radius="0.015" length="0.015">
@@ -133,5 +149,5 @@
   <link name="caster_wheel_support">
     <visual>
-      <origin xyz="0 0 0" rpy="0 0 0"/> <!-- Origen de la visualización del soporte del caster -->
+      <origin xyz="0 0 0" rpy="0 0 0"/>
       <geometry>
         <mesh filename="file://$(find tp1_robot)/meshes/caster_wheel_support.stl"/>
@@ -140,7 +156,7 @@
     </visual>
     <collision>
-      <origin xyz="0 0 0" rpy="0 0 0"/> <!-- Origen de la colisión del soporte del caster -->
-      <geometry>
-        <box size="0.02 0.02 0.02"/> <!-- Tamaño del soporte del caster (x: largo, y: ancho, z: alto) -->
+      <origin xyz="0 0 0" rpy="0 0 0"/>
+      <geometry>
+        <box size="0.02 0.02 0.02"/>
       </geometry>
     </collision>
@@ -186,5 +202,5 @@
       <state_interface name="velocity"/>
     </joint>
-    <!-- Caster no necesita comando, solo estado -->
+    <!-- Caster solo estado -->
     <joint name="caster_wheel_joint">
       <state_interface name="position"/>
@@ -197,7 +213,38 @@
   <gazebo>
     <plugin filename="gz_ros2_control-system" name="gz_ros2_control::GazeboSimROS2ControlPlugin">
-      <parameters>$(find tp1_robot)/config/diffbot_controllers.yaml</parameters>
+      <parameters>$(find tp1_robot)/config/diff_drive_controller.yaml</parameters>
       <robot_sim_type>gz_ros2_control/GazeboSimSystem</robot_sim_type>
+      <control_period>0.01</control_period> <!-- 100 Hz -->
     </plugin>
   </gazebo>
+  <!-- Material base para evitar warnings -->
+  <gazebo reference="base_link">
+    <material>Gazebo/Black</material>
+  </gazebo>
+  <!-- Parámetros físicos generales -->
+  <gazebo reference="left_wheel_joint">
+    <mu1>1.0</mu1>
+    <mu2>1.0</mu2>
+    <fdir1>1 0 0</fdir1>
+    <material>Gazebo/Rubber</material>
+    <kp>1e3</kp>
+    <kd>1e1</kd>
+    <maxContacts>10</maxContacts>
+  </gazebo>
+  <gazebo reference="right_wheel_joint">
+    <mu1>1.0</mu1>
+    <mu2>1.0</mu2>
+    <fdir1>1 0 0</fdir1>
+    <material>Gazebo/Rubber</material>
+    <kp>1e3</kp>
+    <kd>1e1</kd>
+    <maxContacts>10</maxContacts>
+  </gazebo>
+  <gazebo reference="caster_wheel_joint">
+    <mu1>0.8</mu1>
+    <mu2>0.8</mu2>
+    <kp>1e3</kp>
+    <kd>1e1</kd>
+    <maxContacts>10</maxContacts>
+  </gazebo>
 </robot>
