Commit message: Correccion 02092025

File: src/robot_description/urdf/diffbot.urdf.xacro (robot description, xacro)
@@ -6,13 +6,13 @@
   <!-- === Propiedades === -->
   <!-- Definición de propiedades reutilizables: masas, colores, dimensiones de ruedas y caster -->
-  <xacro:property name="chassis_mass" value="0.800" />
+  <xacro:property name="chassis_mass" value="0.800" /> <!-- 800g -->
   <!-- Radio de la rueda en metros -->
-  <xacro:property name="wheel_radius" value="0.035" />
+  <xacro:property name="wheel_radius" value="0.035" /> <!-- 70mm de diámetro = 35mm de radio -->
   <!-- Ancho de la rueda en metros -->
-  <xacro:property name="wheel_width" value="0.025" />
+  <xacro:property name="wheel_width" value="0.025" /> <!-- 25mm de ancho -->
   <!-- Ancho entre ruedas en metros -->
-  <xacro:property name="wheel_separation" value="0.135" />
+  <xacro:property name="wheel_separation" value="0.100" /> <!-- 100mm de ancho del chasis -->
   <!-- Separación entre ruedas en metros -->
-  <xacro:property name="caster_origin_xyz" value="-0.075 0 -0.0075" />
+  <xacro:property name="caster_origin_xyz" value="-0.075 0 -0.0075" /> <!-- Posición del caster respecto al chasis -->
   <!-- Posición del caster respecto al chasis -->
   <xacro:property name="base_elevation" value="0.055" />
@@ -20,5 +20,4 @@
   <xacro:property name="wheel_color" value="silver" />
   <xacro:property name="caster_color" value="orange" />
-  <xacro:property name="wheelSeparation" value="0.13" />
   <!-- ======================= -->
   <!-- === Includes === -->
@@ -47,8 +46,8 @@
       <origin xyz="0 0 0" rpy="0 0 0" />
       <geometry>
-        <box size="0.195 0.1 0.05" />
-      </geometry>
-    </collision>
-    <xacro:inertial_box mass="0.8" x="0.195" y="0.100" z="0.05">
+        <box size="0.195 0.1 0.005" />
+      </geometry>
+    </collision>
+    <xacro:inertial_box mass="0.8" x="0.195" y="0.100" z="0.005">
       <origin xyz="0 0 0.0525" rpy="0 0 0" />
     </xacro:inertial_box>
@@ -81,5 +80,5 @@
         <material name="${wheel_color}" />
       </collision>
-      <xacro:inertial_cylinder mass="0.150" radius="${wheel_radius}" length="${wheel_width}">
+      <xacro:inertial_cylinder mass="0.150" radius="${wheel_radius}" length="${wheel_width}"> <!-- 150g -->
         <origin xyz="0 0 0" rpy="0 0 0" />
       </xacro:inertial_cylinder>
@@ -89,6 +88,6 @@
   <!-- === Ruedas y motores === -->
   <!-- Instanciación de ruedas y motores usando las macros -->
-  <xacro:wheel prefix="left" xyz="0.0185  0.05 -0.0175" axis="0 1 0" rpy="0 1.5708 0"/>
-  <xacro:wheel prefix="right" xyz="0.0185 -0.05 -0.0175" axis="0 -1 0" rpy="0 1.5708 3.14159"/>
+  <xacro:wheel prefix="left" xyz="0.0185  0.05 -0.0175" axis="0 1 0" rpy="0 1.5708 0"/> <!-- Posición rueda izquierda -->
+  <xacro:wheel prefix="right" xyz="0.0185 -0.05 -0.0175" axis="0 -1 0" rpy="0 1.5708 3.14159"/> <!-- Posición rueda derecha -->
   <!-- Motores -->
   <xacro:motor prefix="left" chassis_width="0.1" reflect="false" />
@@ -115,9 +114,8 @@
       <origin xyz="0 0 0.0045" rpy="0 0 0" />
       <geometry>
-        <!--<box size="0.05 0.05 0.01"/>-->
-        <box size="0.033 0.039 0.016" />
-      </geometry>
-    </collision>
-    <xacro:inertial_box mass="0.020" x="0.032" y="0.038" z="0.015">
+        <box size="0.032 0.038 0.015" />
+      </geometry>
+    </collision>
+    <xacro:inertial_box mass="0.020" x="0.032" y="0.038" z="0.015"> <!-- 20g -->
       <origin xyz="0 0 0" rpy="0 0 0" />
     </xacro:inertial_box>
@@ -127,5 +125,5 @@
     <parent link="caster_wheel_support" />
     <child link="caster_wheel" />
-    <origin xyz="-0.015 0 -0.020" rpy="0 0 0" />
+    <origin xyz="-0.015 0 -0.020" rpy="0 0 0" /> <!-- Posición de la rueda giratoria respecto al soporte -->
     <axis xyz="0 1 0" />
   </joint>
@@ -145,9 +143,9 @@
       <origin xyz="0 0 -0.007" rpy="0 0 0" />
       <geometry>
-        <cylinder radius="0.015" length="0.016" />
+        <cylinder radius="0.0075" length="0.015" />
       </geometry>
     </collision>
     <!-- Inercia orientada correctamente -->
-    <xacro:inertial_cylinder mass="0.150" radius="0.015" length="0.016">
+    <xacro:inertial_cylinder mass="0.010" radius="0.0075" length="0.015"> <!-- 10g, 15mm diámetro = 7.5mm radio -->
       <origin xyz="0 0 0" rpy="0 0 0" />
     </xacro:inertial_cylinder>
@@ -157,5 +155,5 @@
     <parent link="base_link" />
     <child link="caster_wheel_support" />
-    <origin xyz="-0.075 0 -0.015" rpy="0 0 0" />
+    <origin xyz="-0.075 0 -0.015" rpy="0 0 0" /> <!-- Posición del soporte de la rueda giratoria -->
     <axis xyz="0 0 1" />
   </joint>
@@ -171,9 +169,8 @@
       <origin xyz="0 0 0" rpy="0 0 0" />
       <geometry>
-        <!--<box size="0.02 0.02 0.02"/>-->
-        <box size="0.033 0.039 0.016" />
-      </geometry>
-    </collision>
-    <xacro:inertial_box mass="0.02" x="0.033" y="0.025" z="0.025">
+        <box size="0.033 0.025 0.025" />
+      </geometry>
+    </collision>
+    <xacro:inertial_box mass="0.020" x="0.033" y="0.025" z="0.025"> <!-- 20g -->
       <origin xyz="0 0 0" rpy="0 0 0" />
     </xacro:inertial_box>

File: src/robot_description/urdf/motor.xacro (robot description, xacro)
@@ -4,8 +4,8 @@
     <xacro:macro name="motor" params="prefix chassis_width:=0 reflect:=false">
         <!-- Parámetros -->
-        <xacro:property name="motor_mass" value="0.1"/>
-        <xacro:property name="motor_x_size" value="0.07"/>
-        <xacro:property name="motor_y_size" value="0.0188"/>
-        <xacro:property name="motor_z_size" value="0.0225"/>
+        <xacro:property name="motor_mass" value="0.1"/> <!-- 100g -->
+        <xacro:property name="motor_x_size" value="0.07"/> <!-- 70mm -->
+        <xacro:property name="motor_y_size" value="0.0188"/> <!-- 18.8mm -->
+        <xacro:property name="motor_z_size" value="0.0225"/> <!-- 22.5mm -->
         <xacro:property name="motor_x_offset" value="0.0015"/>
         <xacro:property name="motor_y_offset" value="0.0216"/>
