Commit message: 08-09-2025-V3

File: diffbot_description/urdf/diffbot.urdf.xacro (robot description, xacro)
@@ -23,6 +23,6 @@
   <!-- === Includes === -->
   <!-- Inclusión de archivos xacro auxiliares para macros de inercia y motor -->
-  <xacro:include filename="$(find robot_description)/urdf/inertial_macros.xacro" />
-  <xacro:include filename="$(find robot_description)/urdf/motor.xacro" />
+  <xacro:include filename="$(find diffbot_description)/urdf/inertial_macros.xacro" />
+  <xacro:include filename="$(find diffbot_description)/urdf/motor.xacro" />
   <link name="base_footprint" />
   <joint name="base_joint" type="fixed">
@@ -38,5 +38,5 @@
       <origin xyz="0 0 0" rpy="0 0 0" />
       <geometry>
-        <mesh filename="file://$(find robot_description)/meshes/chassis.stl"/>
+        <mesh filename="file://$(find diffbot_description)/meshes/chassis.stl"/>
       </geometry>
       <material name="${base_color}" />
@@ -68,5 +68,5 @@
         <origin xyz="0 0 0" rpy="1.5708 0 0" />
         <geometry>
-          <mesh filename="file://$(find robot_description)/meshes/wheel.stl"/>
+          <mesh filename="file://$(find diffbot_description)/meshes/wheel.stl"/>
         </geometry>
         <material name="${wheel_color}" />
@@ -107,5 +107,5 @@
       <origin xyz="0 0 0.0045" rpy="0 0 0" />
       <geometry>
-        <mesh filename="file://$(find robot_description)/meshes/caster_base.stl" />
+        <mesh filename="file://$(find diffbot_description)/meshes/caster_base.stl" />
       </geometry>
       <material name="${caster_color}" />
@@ -135,5 +135,5 @@
       <!--1.5708-->
       <geometry>
-        <mesh filename="file://$(find robot_description)/meshes/caster_wheel.stl" />
+        <mesh filename="file://$(find diffbot_description)/meshes/caster_wheel.stl" />
       </geometry>
       <material name="${caster_color}" />
@@ -162,5 +162,5 @@
       <origin xyz="0 0 0" rpy="0 0 0" />
       <geometry>
-        <mesh filename="file://$(find robot_description)/meshes/caster_wheel_support.stl" />
+        <mesh filename="file://$(find diffbot_description)/meshes/caster_wheel_support.stl" />
       </geometry>
       <material name="${caster_color}" />

File: diffbot_description/urdf/motor.xacro (robot description, xacro)
@@ -21,8 +21,8 @@
                 <geometry>
                     <xacro:if value="${reflect}">
-                        <mesh filename="file://$(find robot_description)/meshes/motor.stl" scale="1 -1 1"/>
+                        <mesh filename="file://$(find diffbot_description)/meshes/motor.stl" scale="1 -1 1"/>
                     </xacro:if>
                     <xacro:unless value="${reflect}">
-                        <mesh filename="file://$(find robot_description)/meshes/motor.stl"/>
+                        <mesh filename="file://$(find diffbot_description)/meshes/motor.stl"/>
                     </xacro:unless>
                 </geometry>

Commit message: 08-09-2025-V7

File: diffbot_description/urdf/diffbot.urdf.xacro (robot description, xacro)
@@ -25,10 +25,4 @@
   <xacro:include filename="$(find diffbot_description)/urdf/inertial_macros.xacro" />
   <xacro:include filename="$(find diffbot_description)/urdf/motor.xacro" />
-  <link name="base_footprint" />
-  <joint name="base_joint" type="fixed">
-    <parent link="base_footprint" />
-    <child link="base_link" />
-    <origin xyz="0 0 ${base_elevation}" rpy="0 0 0" />
-  </joint>
   <!-- ======================= -->
   <!-- === Chasis del robot === -->

Commit message: 16-09-2025-V1

File: diffbot_description/urdf/diffbot.urdf.xacro (robot description, xacro)
@@ -17,11 +17,13 @@
   <!-- Posición del caster respecto al chasis -->
   <xacro:property name="base_elevation" value="0.055" />
-  <xacro:property name="base_color" value="green" />
+  <!-- Colores definidos en materials.xacro -->
+  <!-- <xacro:property name="base_color" value="green" />
   <xacro:property name="wheel_color" value="silver" />
-  <xacro:property name="caster_color" value="orange" />
+  <xacro:property name="caster_color" value="orange" /> -->
   <!-- ======================= -->
   <!-- === Includes === -->
   <!-- Inclusión de archivos xacro auxiliares para macros de inercia y motor -->
   <xacro:include filename="$(find diffbot_description)/urdf/inertial_macros.xacro" />
+  <!-- <xacro:include filename="$(find diffbot_description)/urdf/materials.xacro" /> -->
   <xacro:include filename="$(find diffbot_description)/urdf/motor.xacro" />
   <!-- ======================= -->
@@ -34,6 +36,8 @@
         <mesh filename="file://$(find diffbot_description)/meshes/chassis.stl"/>
       </geometry>
-      <material name="${base_color}" />
-      <!-- Colo que se visualiza en RViz-->
+      <material name="chassis_green">
+        <color rgba="0.0 0.8 0.0 1.0"/>
+      </material>
+      <!-- Color que se visualiza en RViz-->
     </visual>
     <collision>
@@ -64,6 +68,8 @@
           <mesh filename="file://$(find diffbot_description)/meshes/wheel.stl"/>
         </geometry>
-        <material name="${wheel_color}" />
-        <!-- Colo que se visualiza en RViz-->
+        <material name="wheel_silver">
+          <color rgba="0.79 0.82 0.93 1"/>
+        </material>
+        <!-- Color que se visualiza en RViz-->
       </visual>
       <collision>
@@ -72,5 +78,7 @@
           <cylinder radius="${wheel_radius}" length="${wheel_width}"/>
         </geometry>
-        <material name="${wheel_color}" />
+        <material name="wheel_silver_collision">
+          <color rgba="0.79 0.82 0.93 1"/>
+        </material>
       </collision>
       <xacro:inertial_cylinder mass="0.150" radius="${wheel_radius}" length="${wheel_width}"> <!-- 150g -->
@@ -103,5 +111,7 @@
         <mesh filename="file://$(find diffbot_description)/meshes/caster_base.stl" />
       </geometry>
-      <material name="${caster_color}" />
+      <material name="caster_orange">
+        <color rgba="1 0.3 0.1 1"/>
+      </material>
     </visual>
     <collision>
@@ -131,5 +141,7 @@
         <mesh filename="file://$(find diffbot_description)/meshes/caster_wheel.stl" />
       </geometry>
-      <material name="${caster_color}" />
+      <material name="caster_wheel_orange">
+        <color rgba="1 0.3 0.1 1"/>
+      </material>
     </visual>
     <collision>
@@ -146,5 +158,5 @@
   </link>
   <!-- Soporte de la rueda loca -->
-  <joint name="caster_support_joint" type="continuous">
+  <joint name="caster_wheel_support_joint" type="continuous">
     <parent link="base_link" />
     <child link="caster_wheel_support" />
@@ -158,5 +170,7 @@
         <mesh filename="file://$(find diffbot_description)/meshes/caster_wheel_support.stl" />
       </geometry>
-      <material name="${caster_color}" />
+      <material name="caster_support_orange">
+        <color rgba="1 0.3 0.1 1"/>
+      </material>
     </visual>
     <collision>
@@ -187,4 +201,10 @@
       <state_interface name="velocity" />
     </joint>
+    <joint name="caster_wheel_joint">
+      <state_interface name="position" />
+    </joint>
+    <joint name="caster_wheel_support_joint">
+      <state_interface name="position" />
+    </joint>
   </ros2_control>
   <gazebo>
@@ -193,3 +213,12 @@
     </plugin>
   </gazebo>
+  <!-- Plugin de Lidar para gazebo
+  <gazebo>
+    <plugin
+      filename="gz-sim-sensors-system"
+      name="gz::sim::systems::Sensors">
+      <render_engine>ogre2</render_engine>
+    </plugin>
+  </gazebo>
+  -->
 </robot>

File: diffbot_description/urdf/motor.xacro (robot description, xacro)
@@ -27,5 +27,7 @@
                     </xacro:unless>
                 </geometry>
-                <material name="blue"/>
+                <material name="motor_blue">
+                    <color rgba="0.0 0.0 0.8 1.0"/>
+                </material>
             </visual>
             <!-- Colisión -->

Commit message: 16-09-2025-V3

File: diffbot_description/urdf/diffbot.urdf.xacro (robot description, xacro)
@@ -146,6 +146,7 @@
     </visual>
     <collision>
-      <!-- Misma rotación para colisión -->
-      <origin xyz="0 0 -0.007" rpy="0 0 0" />
+      <!-- Ajustado para evitar que la rueda esté por debajo del suelo -->
+      <!-- -0.007 -->
+      <origin xyz="0 0 -0.0075" rpy="0 0 0" />
       <geometry>
         <cylinder radius="0.0075" length="0.015" />

Commit message: 16-09-2025-V4

File: diffbot_description/urdf/diffbot.urdf.xacro (robot description, xacro)
@@ -214,5 +214,79 @@
     </plugin>
   </gazebo>
-  <!-- Plugin de Lidar para gazebo
+  <!-- ================================== SENSORES =============================================-->
+    <!-- ================= IMU COMENTADA =================
+  <link name="imu_link">
+    <xacro:dummy_inertial />
+  </link>
+  <joint name="imu_joint" type="fixed">
+    <parent link="base_link"/>
+    <child link="imu_link"/>
+    <origin xyz="0 0 0.1" rpy="0 0 0"/>
+  </joint>
+  <gazebo reference="imu_link">
+    <sensor name="imu" type="imu">
+      <plugin name="gz::sim::systems::Imu" filename="gz-sim-imu-system">
+        <always_on>true</always_on>
+        <update_rate>100</update_rate>
+        <topic>/imu/data</topic>
+        <visualize>true</visualize>
+      </plugin>
+      <imu>
+        <linear_acceleration>
+          <x>
+            <noise type="gaussian">
+              <mean>0.020</mean>
+              <stddev>0.0016</stddev>
+            </noise>
+          </x>
+          <y>
+            <noise type="gaussian">
+              <mean>0.020</mean>
+              <stddev>0.0016</stddev>
+            </noise>
+          </y>
+          <z>
+            <noise type="gaussian">
+              <mean>0.020</mean>
+              <stddev>0.0019</stddev>
+            </noise>
+          </z>
+        </linear_acceleration>
+        <angular_velocity>
+          <x>
+            <noise type="gaussian">
+              <mean>0.0174533</mean>
+              <stddev>0.00174533</stddev>
+            </noise>
+          </x>
+          <y>
+            <noise type="gaussian">
+              <mean>0.0174533</mean>
+              <stddev>0.00174533</stddev>
+            </noise>
+          </y>
+          <z>
+            <noise type="gaussian">
+              <mean>0.0174533</mean>
+              <stddev>0.00174533</stddev>
+            </noise>
+          </z>
+        </angular_velocity>
+      </imu>
+    </sensor>
+  </gazebo>
+================= FIN IMU COMENTADA ================= -->
+  <!-- Link del sensor LiDAR -->
+  <link name="lidar_link">
+    <!-- Inercial ,no funciona dummy -->
+    <xacro:dummy_inertial />
+  </link>
+  <!-- Joint fijo entre base_link y lidar_link -->
+  <joint name="lidar_joint" type="fixed">
+    <parent link="base_link"/>
+    <child link="lidar_link"/>
+    <origin xyz="0 0 0.15" rpy="0 0 0"/>
+  </joint>
+  <!-- PLUGGIN VALIDO PARA LIDAR Y OTROS SENSORES, SIN COSAS RARAS-->
   <gazebo>
     <plugin
@@ -222,4 +296,32 @@
     </plugin>
   </gazebo>
-  -->
+<!-- Sensor LiDAR en Gazebo -->
+  <gazebo reference="lidar_link">
+    <sensor name="lidar" type="gpu_lidar">
+      <always_on>true</always_on>
+      <update_rate>10</update_rate>
+      <topic>/scan</topic>
+      <visualize>true</visualize>
+      <lidar>
+        <scan>
+          <horizontal>
+            <samples>3200</samples>
+            <min_angle>-3.14159</min_angle>
+            <max_angle>3.14159</max_angle>
+            <resolution>1</resolution>
+          </horizontal>
+        </scan>
+        <range>
+          <min>0.05</min>
+          <max>15.0</max>
+          <resolution>0.01</resolution>
+        </range>
+        <noise>
+          <type>gaussian</type>
+          <mean>0.0</mean>
+          <stddev>0.03</stddev>
+        </noise>
+      </lidar>
+    </sensor>
+  </gazebo>
 </robot>
