Commit message: 24-09-2025-V6

File: diffbot_description/urdf/diffbot.urdf.xacro (robot description, xacro)
@@ -1,28 +1,38 @@
 <?xml version="1.0"?>
+<!--
+  URDF/Xacro del robot DiffBot - Robot diferencial educativo
+  Este archivo define un robot móvil diferencial con:
+  - Chasis principal con ruedas motrices
+  - Rueda loca (caster) para estabilidad
+  - Sensores: Cámara, LiDAR e IMU
+  - Configuración completa para simulación en Gazebo
+  Autor: [Tu nombre]
+  Fecha: [Fecha actual]
+  Versión: 1.0
+-->
 <robot name="diffbot"
   xmlns:xacro="http://www.ros.org/wiki/xacro"
   xmlns:gazebo="http://www.gazebosim.org/schema/gazebo_urdf">
   <!-- ======================= -->
-  <!-- === Propiedades === -->
-  <!-- Parámetros reutilizables -->
-  <xacro:property name="chassis_mass" value="0.8"/>
-  <xacro:property name="chassis_length" value="0.195"/>
-  <xacro:property name="chassis_width" value="0.1"/>
-  <xacro:property name="chassis_height" value="0.005"/>
-  <xacro:property name="wheel_radius" value="0.035"/>
-  <xacro:property name="wheel_separation" value="0.135"/>
-  <!-- Colores definidos en materials.xacro -->
-  <!-- <xacro:property name="base_color" value="green" />
-  <xacro:property name="wheel_color" value="silver" />
-  <xacro:property name="caster_color" value="orange" /> -->
-  <!-- ======================= -->
-  <!-- === Includes === -->
-  <!-- Inclusión de archivos xacro auxiliares para macros de inercia y motor -->
-  <xacro:include filename="$(find diffbot_description)/urdf/materials.xacro" />
-  <xacro:include filename="$(find diffbot_description)/urdf/inertial_macros.xacro" />
-  <xacro:include filename="$(find diffbot_description)/urdf/motor.xacro" />
-  <!-- ======================= -->
-  <!-- === Chasis del robot === -->
-  <!-- Link principal del robot: el chasis -->
+  <!-- === PROPIEDADES === -->
+  <!-- Parámetros físicos reutilizables del robot -->
+  <!-- Propiedades del chasis -->
+  <xacro:property name="chassis_mass" value="0.8"/>        <!-- Masa del chasis: 800g -->
+  <xacro:property name="chassis_length" value="0.195"/>    <!-- Longitud: 19.5 cm -->
+  <xacro:property name="chassis_width" value="0.1"/>       <!-- Ancho: 10 cm -->
+  <xacro:property name="chassis_height" value="0.005"/>    <!-- Altura: 5 mm -->
+  <!-- Propiedades de las ruedas -->
+  <xacro:property name="wheel_radius" value="0.035"/>      <!-- Radio de rueda: 3.5 cm -->
+  <xacro:property name="wheel_separation" value="0.135"/>  <!-- Separación entre ruedas: 13.5 cm -->
+  <!-- Nota: Los colores están definidos en materials.xacro -->
+  <!-- ======================= -->
+  <!-- === ARCHIVOS INCLUIDOS === -->
+  <!-- Inclusión de archivos xacro auxiliares -->
+  <xacro:include filename="$(find diffbot_description)/urdf/materials.xacro" />      <!-- Definiciones de colores -->
+  <xacro:include filename="$(find diffbot_description)/urdf/inertial_macros.xacro" /> <!-- Macros para cálculo de inercias -->
+  <xacro:include filename="$(find diffbot_description)/urdf/motor.xacro" />           <!-- Configuración de motores -->
+  <!-- ======================= -->
+  <!-- === CHASIS PRINCIPAL === -->
+  <!-- Link base del robot (referencia principal) -->
   <link name="base_link">
     <visual>
@@ -31,9 +41,8 @@
         <mesh filename="file://$(find diffbot_description)/meshes/chassis.stl"/>
       </geometry>
-      <material name="chassis_green">
-        <color rgba="0.0 0.8 0.0 1.0"/>
-      </material>
-      <!-- Color que se visualiza en RViz-->
-    </visual>
+      <material name="green"/>
+      <!-- Color verde para visualización en RViz/Gazebo -->
+    </visual>
+    <!-- Geometría de colisión (caja simplificada) -->
     <collision>
       <origin xyz="0 0 0" rpy="0 0 0" />
@@ -42,4 +51,5 @@
       </geometry>
     </collision>
+    <!-- Propiedades inerciales calculadas automáticamente -->
     <xacro:inertial_box mass="${chassis_mass}" x="${chassis_length}" y="${chassis_width}" z="0.00">
       <origin xyz="0 0 0" rpy="0 0 0" />
@@ -47,29 +57,34 @@
   </link>
   <!-- ======================= -->
-  <!-- === Macro para ruedas === -->
-  <!-- Macro reutilizable para definir una rueda y su joint asociado. Parametrizado por radio y
-  separación. -->
+  <!-- === MACRO PARA RUEDAS === -->
+  <!-- Macro reutilizable para definir ruedas motrices -->
+  <!-- Parámetros: prefix (izq/der), xyz (posición), axis (eje rotación), rpy (orientación) -->
   <xacro:macro name="wheel" params="prefix xyz axis rpy">
+    <!-- Joint continuo para rotación libre de la rueda -->
     <joint name="${prefix}_wheel_joint" type="continuous">
       <parent link="base_link" />
       <child link="${prefix}_wheel_link" />
-      <origin xyz="${xyz}" rpy="${rpy}" />
-      <axis xyz="${axis}" />
+      <origin xyz="${xyz}" rpy="${rpy}" />     <!-- Posición y orientación de la rueda -->
+      <axis xyz="${axis}" />                   <!-- Eje de rotación -->
     </joint>
+    <!-- Link de la rueda -->
     <link name="${prefix}_wheel_link">
+      <!-- Geometría visual (mesh 3D) -->
       <visual>
-        <origin xyz="0 -0.020 0" rpy="1.5708 0 0" />
+        <origin xyz="0 -0.020 0" rpy="1.5708 0 0" />  <!-- Ajuste de posición y rotación -->
         <geometry>
           <mesh filename="file://$(find diffbot_description)/meshes/wheel.stl"/>
         </geometry>
-        <material name="dark_grey"/>
+        <material name="dark_grey"/>                   <!-- Color gris oscuro -->
       </visual>
+      <!-- Geometría de colisión (cilindro simplificado) -->
       <collision>
         <origin xyz="0 -0.020 0" rpy="1.5708 0 0" />
         <geometry>
-          <cylinder radius="${wheel_radius}" length="0.025"/>
+          <cylinder radius="${wheel_radius}" length="0.025"/>  <!-- Radio y grosor de rueda -->
         </geometry>
         <material name="dark_grey"/>
       </collision>
+      <!-- Propiedades inerciales de cilindro (masa: 150g) -->
       <xacro:inertial_cylinder mass="0.150" radius="${wheel_radius}" length="0.025">
         <origin xyz="0 0 0" rpy="0 0 0" />
@@ -78,16 +93,20 @@
   </xacro:macro>
   <!-- ======================= -->
-  <!-- === Ruedas y motores === -->
-  <!-- Instanciación de ruedas y motores usando las macros -->
+  <!-- === INSTANCIACIÓN DE RUEDAS Y MOTORES === -->
+  <!-- Creación de ruedas izquierda y derecha con sus respectivos motores -->
+  <!-- Rueda izquierda -->
   <xacro:wheel prefix="left" xyz="0.0185  ${wheel_separation/2} -0.0175" axis="0 1 0" rpy="0 1.5708 0"/>
+  <!-- Rueda derecha -->
   <xacro:wheel prefix="right" xyz="0.0185 -${wheel_separation/2} -0.0175" axis="0 -1 0" rpy="0 1.5708 3.14159"/>
-  <!-- Motores -->
-  <xacro:motor prefix="left" chassis_width="${chassis_width}" reflect="false"/>
-  <xacro:motor prefix="right" chassis_width="${chassis_width}" reflect="true"/>
-  <!-- ======================= -->
-  <!-- === Caster (rueda loca) === -->
-  <!-- Definición del caster y sus componentes -->
-  <!-- BASE FIJA -->
+  <!-- Motores para tracción diferencial -->
+  <xacro:motor prefix="left" chassis_width="${chassis_width}" reflect="false"/>   <!-- Motor izquierdo -->
+  <xacro:motor prefix="right" chassis_width="${chassis_width}" reflect="true"/>    <!-- Motor derecho -->
+  <!-- ======================= -->
+  <!-- === CASTER (RUEDA LOCA) === -->
+  <!-- Rueda loca trasera para estabilidad del robot -->
+  <!-- BASE FIJA DEL CASTER -->
+  <!-- Link de la base del caster (parte fija) -->
   <link name="caster_base">
+    <!-- Geometría visual (mesh 3D) -->
     <visual>
       <origin xyz="0 0 0.0045" rpy="0 0 0" />
@@ -95,47 +114,51 @@
         <mesh filename="file://$(find diffbot_description)/meshes/caster_base.stl" />
       </geometry>
-      <material name="caster_orange">
-        <color rgba="1 0.3 0.1 1"/>
-      </material>
-    </visual>
+      <material name="orange"/>              <!-- Color naranja -->
+    </visual>
+    <!-- Geometría de colisión (caja simplificada) -->
     <collision>
       <origin xyz="0 0 0.0045" rpy="0 0 0" />
       <geometry>
-        <box size="0.032 0.038 0.015" />
-      </geometry>
-    </collision>
+        <box size="0.032 0.038 0.015" />          <!-- Dimensiones de la base -->
+      </geometry>
+    </collision>
+    <!-- Propiedades inerciales (masa: 20g) -->
     <xacro:inertial_box mass="0.02" x="0.032" y="0.038" z="0.015">
       <origin xyz="0 0 0" rpy="0 0 0" />
     </xacro:inertial_box>
   </link>
+  <!-- Joint fijo que conecta la base del caster al chasis -->
   <joint name="caster_base_joint" type="fixed">
-    <origin xyz="-0.075 0 -0.001" rpy="0 0 0"/>
+    <origin xyz="-0.075 0 -0.001" rpy="0 0 0"/>  <!-- Posición trasera del robot -->
     <parent link="base_link"/>
     <child link="caster_base"/>
   </joint>
-  <!-- RUEDA MOVIL  -->
+  <!-- RUEDA MÓVIL DEL CASTER -->
+  <!-- Link de la rueda loca (gira libremente) -->
   <link name="caster_wheel">
-    <visual>
-      <!-- Rotamos el cilindro 90° alrededor del eje X para que su eje de giro sea el eje Y -->
-      <origin xyz="0 0 0" rpy="0 0 0" />
-      <!--1.5708-->
+    <!-- Geometría visual (mesh 3D) -->
+    <visual>
+      <origin xyz="0 0 0" rpy="0 0 0" />
       <geometry>
         <mesh filename="file://$(find diffbot_description)/meshes/caster_wheel.stl" />
       </geometry>
-      <material name="caster_wheel_orange">
-        <color rgba="1 0.3 0.1 1"/>
-      </material>
-    </visual>
+      <material name="orange"/>              <!-- Color naranja -->
+    </visual>
+    <!-- Geometría de colisión (cilindro) -->
     <collision>
       <origin xyz="0 0 -0.007" rpy="0 0 0" />
       <geometry>
-        <cylinder radius="0.015" length="0.016" />
-      </geometry>
-    </collision>
+        <cylinder radius="0.015" length="0.016" />  <!-- Radio: 1.5cm, Grosor: 1.6cm -->
+      </geometry>
+    </collision>
+    <!-- Propiedades inerciales de cilindro (masa: 10g) -->
     <xacro:inertial_cylinder mass="0.01" radius="0.015" length="0.016">
       <origin xyz="0 0 0" rpy="0 0 0" />
     </xacro:inertial_cylinder>
   </link>
+  <!-- SOPORTE DE LA RUEDA CASTER -->
+  <!-- Link del soporte que permite rotación vertical -->
   <link name="caster_wheel_support">
+    <!-- Geometría visual (mesh 3D) -->
     <visual>
       <origin xyz="0 0 0" rpy="0 0 0" />
@@ -143,127 +166,81 @@
         <mesh filename="file://$(find diffbot_description)/meshes/caster_wheel_support.stl" />
       </geometry>
-      <material name="caster_support_orange">
-        <color rgba="1 0.3 0.1 1"/>
-      </material>
-    </visual>
-    <collision>
-      <origin xyz="0 0 0" rpy="0 0 0" />
-      <geometry>
-        <box size="0.033 0.025 0.025" />
-      </geometry>
-    </collision>
+      <material name="orange"/>              <!-- Color naranja -->
+    </visual>
+    <!-- Geometría de colisión (caja) -->
+    <collision>
+      <origin xyz="0 0 0" rpy="0 0 0" />
+      <geometry>
+        <box size="0.033 0.025 0.025" />          <!-- Dimensiones del soporte -->
+      </geometry>
+    </collision>
+    <!-- Propiedades inerciales (masa: 20g) -->
     <xacro:inertial_box mass="0.02" x="0.033" y="0.025" z="0.025">
       <origin xyz="0 0 0" rpy="0 0 0" />
     </xacro:inertial_box>
   </link>
+  <!-- Joint continuo para rotación vertical del soporte (eje Z) -->
   <joint name="caster_wheel_support_joint" type="continuous">
     <origin xyz="0 0 -0.015" rpy="0 0 0"/>
     <parent link="caster_base"/>
     <child link="caster_wheel_support"/>
-    <axis xyz="0 0 1"/>
-  </joint>
-  <!-- Rueda loca -->
+    <axis xyz="0 0 1"/>                          <!-- Rotación alrededor del eje Z -->
+  </joint>
+  <!-- Joint continuo para rotación de la rueda loca (eje Y) -->
   <joint name="caster_wheel_joint" type="continuous">
     <origin xyz="-0.015 0 -0.020" rpy="0 0 0"/>
     <parent link="caster_wheel_support"/>
     <child link="caster_wheel"/>
-    <axis xyz="0 1 0"/>
-  </joint>
-  <!-- Configuración de ros2_control para la interfaz de hardware -->
-  <!-- El nombre "GazeboSystem" y el tipo "system" son estándar para la integración con Gazebo. -->
+    <axis xyz="0 1 0"/>                          <!-- Rotación alrededor del eje Y -->
+  </joint>
+  <!-- ======================= -->
+  <!-- === CONFIGURACIÓN ROS2_CONTROL === -->
+  <!-- Interfaz de hardware para control de motores en simulación -->
   <ros2_control name="GazeboSystem" type="system">
     <hardware>
-      <!-- Plugin de Gazebo para ROS 2 Control -->
+      <!-- Plugin de Gazebo para integración con ROS 2 Control -->
       <plugin>gz_ros2_control/GazeboSimSystem</plugin>
     </hardware>
+    <!-- Configuración del joint de la rueda izquierda -->
     <joint name="left_wheel_joint">
-      <command_interface name="velocity" />
-      <state_interface name="position" />
-      <state_interface name="velocity" />
+      <command_interface name="velocity" />      <!-- Interfaz de comando: velocidad angular -->
+      <state_interface name="position" />        <!-- Estado: posición angular -->
+      <state_interface name="velocity" />        <!-- Estado: velocidad angular -->
     </joint>
+    <!-- Configuración del joint de la rueda derecha -->
     <joint name="right_wheel_joint">
-      <command_interface name="velocity" />
-      <state_interface name="position" />
-      <state_interface name="velocity" />
+      <command_interface name="velocity" />      <!-- Interfaz de comando: velocidad angular -->
+      <state_interface name="position" />        <!-- Estado: posición angular -->
+      <state_interface name="velocity" />        <!-- Estado: velocidad angular -->
     </joint>
+    <!-- Configuración del joint de la rueda caster (solo lectura) -->
     <joint name="caster_wheel_joint">
-      <state_interface name="position" />
+      <state_interface name="position" />        <!-- Estado: posición angular -->
     </joint>
+    <!-- Configuración del joint del soporte caster (solo lectura) -->
     <joint name="caster_wheel_support_joint">
-      <state_interface name="position" />
+      <state_interface name="position" />        <!-- Estado: posición angular -->
     </joint>
   </ros2_control>
+  <!-- Plugin de Gazebo para ros2_control -->
   <gazebo>
-    <!--<plugin filename="gz_ros2_control-system" name="gz_ros2_control::GazeboSimROS2ControlPlugin">-->
+    <!-- Plugin que conecta ros2_control con la simulación de Gazebo -->
     <plugin filename="libgz_ros2_control-system.so" name="gz_ros2_control::GazeboSimROS2ControlPlugin">
+      <!-- Archivo de configuración de controladores -->
       <parameters>$(find diffbot_control)/config/controllers.yaml</parameters>
     </plugin>
   </gazebo>
-  <!-- ================================== SENSORES =============================================-->
-    <!-- ================= IMU COMENTADA =================
-  <link name="imu_link">
-    <xacro:dummy_inertial />
-  </link>
-  <joint name="imu_joint" type="fixed">
-    <parent link="base_link"/>
-    <child link="imu_link"/>
-    <origin xyz="0 0 0.1" rpy="0 0 0"/>
-  </joint>
-  <gazebo reference="imu_link">
-    <sensor name="imu" type="imu">
-      <plugin name="gz::sim::systems::Imu" filename="gz-sim-imu-system">
-        <always_on>true</always_on>
-        <update_rate>100</update_rate>
-        <topic>/imu/data</topic>
-        <visualize>true</visualize>
-      </plugin>
-      <imu>
-        <linear_acceleration>
-          <x>
-            <noise type="gaussian">
-              <mean>0.020</mean>
-              <stddev>0.0016</stddev>
-            </noise>
-          </x>
-          <y>
-            <noise type="gaussian">
-              <mean>0.020</mean>
-              <stddev>0.0016</stddev>
-            </noise>
-          </y>
-          <z>
-            <noise type="gaussian">
-              <mean>0.020</mean>
-              <stddev>0.0019</stddev>
-            </noise>
-          </z>
-        </linear_acceleration>
-        <angular_velocity>
-          <x>
-            <noise type="gaussian">
-              <mean>0.0174533</mean>
-              <stddev>0.00174533</stddev>
-            </noise>
-          </x>
-          <y>
-            <noise type="gaussian">
-              <mean>0.0174533</mean>
-              <stddev>0.00174533</stddev>
-            </noise>
-          </y>
-          <z>
-            <noise type="gaussian">
-              <mean>0.0174533</mean>
-              <stddev>0.00174533</stddev>
-            </noise>
-          </z>
-        </angular_velocity>
-      </imu>
-    </sensor>
-  </gazebo>
-================= FIN IMU COMENTADA ================= -->
-  <!-- ======================= -->
-  <!-- === SENSOR IMU === -->
-  <!-- ======================= -->
+  <!-- ======================= -->
+  <!-- === SENSORES DEL ROBOT === -->
+  <!-- ======================= -->
+  <!-- NOTA: Configuración IMU anterior (comentada para referencia) -->
+  <!--
+    La configuración IMU comentada arriba era una implementación anterior
+    que ha sido reemplazada por la configuración activa más abajo.
+    Se mantiene como referencia para comparación de parámetros.
+  -->
+  <!-- ======================= -->
+  <!-- === SENSOR IMU ACTIVO === -->
+  <!-- Unidad de Medición Inercial para orientación y aceleración -->
   <!-- Link del IMU -->
   <link name="imu_link">
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
Commit message: 24-09-2025-V11

File: diffbot_description/urdf/diffbot.urdf.xacro (robot description, xacro)
@@ -355,4 +355,6 @@
     <!-- Montada al frente y un poco arriba del chasis -->
     <origin xyz="0.08 0.0 0.015" rpy="0 0 0"/>
+    <!-- Inclinar la camara 15° -->
+    <!-- <origin xyz="0.08 0.0 0.015" rpy="0 ${15*(pi/180)} 0"/> -->
     <parent link="base_link"/>
     <child link="cam_link"/>
